File: hardware/NMOS.kicad_sch (KiCad schematic)
At the start: 5 parts, among them Q3 NMOS

Commit message: meow
Parts:
- R34: value R -> 1k
Changed lines of the file:
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@@
 			)
 		)
-		(property "Value" "R"
+		(property "Value" "1k"
 			(at 120.65 68.58 90)
 			(show_name no)
