File: hardware/NMOS.kicad_sch (KiCad schematic)
At the start: 5 parts, among them Q3 NMOS

Commit message: techuri
Parts:
- removed R34: 1k, symbol Device:R
Connections:
- net In: now also C48.1, Q3.2 (G), R35.1
Changed lines of the file:
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@@
 	(wire
 		(pts
-			(xy 107.95 72.39) (xy 116.84 72.39)
+			(xy 107.95 72.39) (xy 124.46 72.39)
 		)
 		(stroke
@@
 					(unit 1)
 				)
-			)
-		)
-	)
-	(symbol
-		(lib_id "Device:R")
-		(at 120.65 72.39 90)
-		(unit 1)
-		(body_style 1)
-		(exclude_from_sim no)
-		(in_bom yes)
-		(on_board yes)
-		(in_pos_files yes)
-		(dnp no)
-		(property "Reference" "R34"
-			(at 120.65 66.04 90)
-			(show_name no)
-			(do_not_autoplace no)
-			(effects
-				(font
-					(size 1.27 1.27)
-				)
-			)
-		)
-		(property "Value" "1k"
-			(at 120.396 72.136 90)
-			(show_name no)
-			(do_not_autoplace no)
-			(effects
-				(font
-					(size 1.27 1.27)
-				)
-			)
-		)
-		(property "Footprint" ""
-			(at 120.65 74.168 90)
-			(hide yes)
-			(show_name no)
-			(do_not_autoplace no)
-			(effects
-				(font
-					(size 1.27 1.27)
-				)
-			)
-		)
-		(property "Datasheet" ""
-			(at 120.65 72.39 0)
-			(hide yes)
-			(show_name no)
-			(do_not_autoplace no)
-			(effects
-				(font
-					(size 1.27 1.27)
-				)
-			)
-		)
-		(property "Description" "Resistor"
-			(at 120.65 72.39 0)
-			(hide yes)
-			(show_name no)
-			(do_not_autoplace no)
-			(effects
-				(font
-					(size 1.27 1.27)
-				)
-			)
-		)
-		(pin "2"
-		)
-		(pin "1"
-		)
-		(instances
-			(project "DEI"
-				(path "/1469f349-54e5-4a37-953e-ac48c70e29b2/2751c2d7-629c-4bb6-8dd2-1a829c053e6c/1052dbcd-ea1d-4c47-90b9-da589e115318"
-					(reference "R58")
-					(unit 1)
-				)
-				(path "/1469f349-54e5-4a37-953e-ac48c70e29b2/2751c2d7-629c-4bb6-8dd2-1a829c053e6c/13a0f7f7-8bab-40a0-b17e-5f7caba758b4"
-					(reference "R37")
-					(unit 1)
-				)
-				(path "/1469f349-54e5-4a37-953e-ac48c70e29b2/2751c2d7-629c-4bb6-8dd2-1a829c053e6c/1a7db479-e739-453a-8d5e-08bdcac73e65"
-					(reference "R61")
-					(unit 1)
-				)
-				(path "/1469f349-54e5-4a37-953e-ac48c70e29b2/2751c2d7-629c-4bb6-8dd2-1a829c053e6c/45570e4c-379f-4a94-bf7b-4e6e661a26d7"
-					(reference "R52")
-					(unit 1)
-				)
-				(path "/1469f349-54e5-4a37-953e-ac48c70e29b2/2751c2d7-629c-4bb6-8dd2-1a829c053e6c/75f5da1c-00c8-446b-8fb1-52f678584a36"
-					(reference "R55")
-					(unit 1)
-				)
-				(path "/1469f349-54e5-4a37-953e-ac48c70e29b2/2751c2d7-629c-4bb6-8dd2-1a829c053e6c/80e0ce96-c72a-437f-9f1a-24ade86bb32b"
-					(reference "R34")
-					(unit 1)
-				)
-				(path "/1469f349-54e5-4a37-953e-ac48c70e29b2/2751c2d7-629c-4bb6-8dd2-1a829c053e6c/8aa22198-d0e5-42a7-9227-03e81c0b7aba"
-					(reference "R64")
-					(unit 1)
-				)
-				(path "/1469f349-54e5-4a37-953e-ac48c70e29b2/2751c2d7-629c-4bb6-8dd2-1a829c053e6c/8e9fd3b0-a079-439d-b991-b5f36c876be8"
-					(reference "R67")
-					(unit 1)
-				)
-				(path "/1469f349-54e5-4a37-953e-ac48c70e29b2/2751c2d7-629c-4bb6-8dd2-1a829c053e6c/9e69b250-54ae-4160-ad7a-79758089623e"
-					(reference "R43")
-					(unit 1)
-				)
-				(path "/1469f349-54e5-4a37-953e-ac48c70e29b2/2751c2d7-629c-4bb6-8dd2-1a829c053e6c/a3734377-21d2-4bfe-ba0f-545a48d42db5"
-					(reference "R40")
-					(unit 1)
-				)
-				(path "/1469f349-54e5-4a37-953e-ac48c70e29b2/2751c2d7-629c-4bb6-8dd2-1a829c053e6c/b7ac561b-2ba1-4cdf-9509-2d2feeeba778"
-					(reference "R46")
-					(unit 1)
-				)
-				(path "/1469f349-54e5-4a37-953e-ac48c70e29b2/2751c2d7-629c-4bb6-8dd2-1a829c053e6c/d3b2881e-e026-460b-b8e3-6473f820ed1b"
-					(reference "R49")
-					(unit 1)
-				)

Commit message: someone please check if i fucked up removing boot
Parts:
- added D14: Blue Status, symbol Device:LED
Connections:
- net Out: now also D14.1 (K); no longer Q3.1 (D), R33.2
- new net: D14.2 (A), Q3.1 (D), R33.2
Other:
- moved on the sheet: Q3, R33
Changed lines of the file:
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@@
 	(paper "A4")
 	(junction
-		(at 114.3 64.77)
+		(at 133.35 72.39)
 		(diameter 0)
 		(color 0 0 0 0)
@@
 		(color 0 0 0 0)
 	)
+	(junction
+		(at 151.13 66.04)
+		(diameter 0)
+		(color 0 0 0 0)
+	)
 	(wire
 		(pts
@@
 	(wire
 		(pts
-			(xy 124.46 72.39) (xy 124.46 76.2)
+			(xy 151.13 66.04) (xy 151.13 63.5)
 		)
 		(stroke
@@
 	(wire
 		(pts
-			(xy 107.95 72.39) (xy 124.46 72.39)
+			(xy 124.46 72.39) (xy 124.46 76.2)
 		)
 		(stroke
@@
 	(wire
 		(pts
-			(xy 114.3 62.23) (xy 114.3 64.77)
+			(xy 133.35 72.39) (xy 143.51 72.39)
 		)
 		(stroke
@@
 	(wire
 		(pts
-			(xy 124.46 72.39) (xy 133.35 72.39)
+			(xy 151.13 77.47) (xy 151.13 85.09)
 		)
 		(stroke
@@
 	(wire
 		(pts
-			(xy 114.3 64.77) (xy 119.38 64.77)
+			(xy 107.95 72.39) (xy 124.46 72.39)
 		)
 		(stroke
@@
 	(wire
 		(pts
-			(xy 107.95 64.77) (xy 114.3 64.77)
+			(xy 170.18 66.04) (xy 179.07 66.04)
 		)
 		(stroke
@@
 		)
 	)
+	(wire
+		(pts
+			(xy 124.46 72.39) (xy 133.35 72.39)
+		)
+		(stroke
+			(width 0)
+			(type default)
+		)
+	)
+	(wire
+		(pts
+			(xy 151.13 66.04) (xy 162.56 66.04)
+		)
+		(stroke
+			(width 0)
+			(type default)
+		)
+	)
+	(wire
+		(pts
+			(xy 151.13 66.04) (xy 151.13 67.31)
+		)
+		(stroke
+			(width 0)
+			(type default)
+		)
+	)
 	(hierarchical_label "Out"
 		(shape output)
-		(at 107.95 64.77 180)
+		(at 179.07 66.04 0)
 		(effects
 			(font
 				(size 1.27 1.27)
 			)
-			(justify right)
+			(justify left)
 		)
 	)
@@
 	(hierarchical_label "GND"
 		(shape output)
-		(at 129.54 64.77 0)
+		(at 151.13 80.01 0)
 		(effects
 			(font
@@
 	(symbol
 		(lib_id "power:GND")
-		(at 129.54 64.77 0)
+		(at 151.13 85.09 0)
 		(unit 1)
 		(body_style 1)
@@
 		(fields_autoplaced yes)
 		(property "Reference" "#PWR014"
-			(at 129.54 71.12 0)
+			(at 151.13 91.44 0)
 			(hide yes)
 			(show_name no)
@@
 		)
 		(property "Value" "GND"
-			(at 129.54 69.85 0)
+			(at 151.13 90.17 0)
 			(hide yes)
 			(show_name no)
@@
 		)
 		(property "Footprint" ""
-			(at 129.54 64.77 0)
+			(at 151.13 85.09 0)
 			(hide yes)
 			(show_name no)
@@
 		)
 		(property "Datasheet" ""
-			(at 129.54 64.77 0)
+			(at 151.13 85.09 0)
 			(hide yes)
 			(show_name no)
@@
 		)
 		(property "Description" "Power symbol creates a global label with name \"GND\" , ground"
-			(at 129.54 64.77 0)
+			(at 151.13 85.09 0)
 			(hide yes)
 			(show_name no)
@@
 	(symbol
 		(lib_id "Simulation_SPICE:NMOS")
-		(at 124.46 67.31 90)
+		(at 148.59 72.39 0)
 		(unit 1)
 		(body_style 1)
@@
 		(fields_autoplaced yes)
 		(property "Reference" "Q3"
-			(at 124.46 58.42 90)
+			(at 157.48 72.39 90)
 			(show_name no)
 			(do_not_autoplace no)
@@
 		)
 		(property "Value" "NMOS"
-			(at 124.46 60.96 90)
+			(at 154.94 72.39 90)
 			(show_name no)
 			(do_not_autoplace no)
@@
 		)
 		(property "Footprint" ""
-			(at 121.92 62.23 0)
+			(at 153.67 69.85 0)
 			(hide yes)
 			(show_name no)
@@
 		)
 		(property "Datasheet" "https://ngspice.sourceforge.io/docs/ngspice-html-manual/manual.xhtml#cha_MOSFETs"
-			(at 137.16 67.31 0)
+			(at 148.59 85.09 0)
 			(hide yes)
 			(show_name no)
@@
 		)
 		(property "Description" "N-MOSFET transistor, drain/source/gate"
-			(at 124.46 67.31 0)
+			(at 148.59 72.39 0)
 			(hide yes)
 			(show_name no)
@@
 		)
 		(property "Sim.Device" "NMOS"
-			(at 141.605 67.31 0)
+			(at 148.59 89.535 0)
 			(hide yes)
 			(show_name no)
@@
 		)
 		(property "Sim.Type" "VDMOS"
-			(at 143.51 67.31 0)
+			(at 148.59 91.44 0)
 			(hide yes)
 			(show_name no)
@@
 		)
 		(property "Sim.Pins" "1=D 2=G 3=S"
-			(at 139.7 67.31 0)
+			(at 148.59 87.63 0)
 			(hide yes)
 			(show_name no)
@@
 	(symbol
 		(lib_id "power:+3.3V")
-		(at 114.3 54.61 0)
+		(at 151.13 55.88 0)
 		(unit 1)
 		(body_style 1)
@@
 		(fields_autoplaced yes)
 		(property "Reference" "#PWR015"
-			(at 114.3 58.42 0)
+			(at 151.13 59.69 0)
 			(hide yes)
 			(show_name no)
@@
 		)
 		(property "Value" "+3.3V"
-			(at 114.3 49.53 0)
+			(at 151.13 50.8 0)
 			(show_name no)
 			(do_not_autoplace no)
@@
 		)
 		(property "Footprint" ""
-			(at 114.3 54.61 0)
+			(at 151.13 55.88 0)
 			(hide yes)
 			(show_name no)
@@
 		)
 		(property "Datasheet" ""
-			(at 114.3 54.61 0)
+			(at 151.13 55.88 0)
 			(hide yes)
 			(show_name no)
@@
 		)
 		(property "Description" "Power symbol creates a global label with name \"+3.3V\""
-			(at 114.3 54.61 0)
+			(at 151.13 55.88 0)
 			(hide yes)
 			(show_name no)
@@
 	(symbol
 		(lib_id "Device:R")
-		(at 114.3 58.42 0)
+		(at 151.13 59.69 0)
 		(unit 1)
 		(body_style 1)
@@
 		(fields_autoplaced yes)
 		(property "Reference" "R33"
-			(at 116.84 57.1499 0)
+			(at 153.67 58.4199 0)
 			(show_name no)
 			(do_not_autoplace no)
@@
 		)
 		(property "Value" "10K"
-			(at 116.84 59.6899 0)
+			(at 153.67 60.9599 0)
 			(show_name no)
 			(do_not_autoplace no)
@@
 		)
 		(property "Footprint" ""
-			(at 112.522 58.42 90)
+			(at 149.352 59.69 90)
 			(hide yes)
 			(show_name no)
@@
 		)
 		(property "Datasheet" ""
-			(at 114.3 58.42 0)
+			(at 151.13 59.69 0)
 			(hide yes)
 			(show_name no)
@@
 		)
 		(property "Description" "Resistor"
-			(at 114.3 58.42 0)
+			(at 151.13 59.69 0)
 			(hide yes)
 			(show_name no)
@@
 					(unit 1)
 				)
+			)
+		)
+	)
+	(symbol
+		(lib_id "Device:LED")
+		(at 166.37 66.04 180)
+		(unit 1)
+		(body_style 1)
+		(exclude_from_sim no)
+		(in_bom yes)
+		(on_board yes)
+		(in_pos_files yes)
+		(dnp no)
+		(fields_autoplaced yes)
+		(property "Reference" "D14"
+			(at 167.9575 58.42 0)
+			(show_name no)
+			(do_not_autoplace no)
+			(effects
+				(font
+					(size 1.27 1.27)
+				)
+			)
+		)
+		(property "Value" "Blue Status"
+			(at 167.9575 60.96 0)
+			(show_name no)
+			(do_not_autoplace no)
+			(effects
+				(font
+					(size 1.27 1.27)
+				)
+			)
+		)
+		(property "Footprint" ""
+			(at 166.37 66.04 0)
+			(hide yes)
+			(show_name no)
+			(do_not_autoplace no)
+			(effects
+				(font
+					(size 1.27 1.27)
+				)
+			)
+		)
+		(property "Datasheet" ""
+			(at 166.37 66.04 0)
+			(hide yes)
+			(show_name no)
+			(do_not_autoplace no)
+			(effects
+				(font
+					(size 1.27 1.27)
+				)
+			)
+		)
+		(property "Description" "Light emitting diode"
+			(at 166.37 66.04 0)
+			(hide yes)
+			(show_name no)
+			(do_not_autoplace no)
+			(effects
+				(font
+					(size 1.27 1.27)
+				)
+			)
+		)
+		(property "Sim.Pins" "1=K 2=A"
+			(at 166.37 66.04 0)
+			(hide yes)
+			(show_name no)
+			(do_not_autoplace no)
+			(effects
+				(font
+					(size 1.27 1.27)
+				)
+			)
+		)
+		(pin "1"
+		)
+		(pin "2"
+		)
+		(instances
+			(project "DEI"
+				(path "/1469f349-54e5-4a37-953e-ac48c70e29b2/2751c2d7-629c-4bb6-8dd2-1a829c053e6c/1052dbcd-ea1d-4c47-90b9-da589e115318"
+					(reference "D27")
+					(unit 1)
+				)
+				(path "/1469f349-54e5-4a37-953e-ac48c70e29b2/2751c2d7-629c-4bb6-8dd2-1a829c053e6c/13a0f7f7-8bab-40a0-b17e-5f7caba758b4"
+					(reference "D15")
+					(unit 1)
+				)
+				(path "/1469f349-54e5-4a37-953e-ac48c70e29b2/2751c2d7-629c-4bb6-8dd2-1a829c053e6c/1a7db479-e739-453a-8d5e-08bdcac73e65"
+					(reference "D28")
+					(unit 1)
+				)
+				(path "/1469f349-54e5-4a37-953e-ac48c70e29b2/2751c2d7-629c-4bb6-8dd2-1a829c053e6c/45570e4c-379f-4a94-bf7b-4e6e661a26d7"
+					(reference "D25")
+					(unit 1)
+				)
+				(path "/1469f349-54e5-4a37-953e-ac48c70e29b2/2751c2d7-629c-4bb6-8dd2-1a829c053e6c/75f5da1c-00c8-446b-8fb1-52f678584a36"
+					(reference "D26")
+					(unit 1)
+				)
+				(path "/1469f349-54e5-4a37-953e-ac48c70e29b2/2751c2d7-629c-4bb6-8dd2-1a829c053e6c/80e0ce96-c72a-437f-9f1a-24ade86bb32b"
+					(reference "D14")
+					(unit 1)
+				)
+				(path "/1469f349-54e5-4a37-953e-ac48c70e29b2/2751c2d7-629c-4bb6-8dd2-1a829c053e6c/8aa22198-d0e5-42a7-9227-03e81c0b7aba"
+					(reference "D29")
+					(unit 1)
+				)
+				(path "/1469f349-54e5-4a37-953e-ac48c70e29b2/2751c2d7-629c-4bb6-8dd2-1a829c053e6c/8e9fd3b0-a079-439d-b991-b5f36c876be8"
+					(reference "D30")
+					(unit 1)
+				)
+				(path "/1469f349-54e5-4a37-953e-ac48c70e29b2/2751c2d7-629c-4bb6-8dd2-1a829c053e6c/9e69b250-54ae-4160-ad7a-79758089623e"
+					(reference "D17")
+					(unit 1)
+				)
+				(path "/1469f349-54e5-4a37-953e-ac48c70e29b2/2751c2d7-629c-4bb6-8dd2-1a829c053e6c/a3734377-21d2-4bfe-ba0f-545a48d42db5"
+					(reference "D16")
+					(unit 1)
+				)
+				(path "/1469f349-54e5-4a37-953e-ac48c70e29b2/2751c2d7-629c-4bb6-8dd2-1a829c053e6c/b7ac561b-2ba1-4cdf-9509-2d2feeeba778"
+					(reference "D23")
+					(unit 1)
+				)
+				(path "/1469f349-54e5-4a37-953e-ac48c70e29b2/2751c2d7-629c-4bb6-8dd2-1a829c053e6c/d3b2881e-e026-460b-b8e3-6473f820ed1b"
+					(reference "D24")
+					(unit 1)
+				)

Commit message: rawr
Parts:
- removed D14: Blue Status, symbol Device:LED
- added D49: Blue Status, symbol Device:LED
- added R97: 1k, symbol Device:R
- renumbered C48 to C64, Q3 to Q17, R35 to R98, R33 to R99
Connections:
- net GND: now also D49.1 (K)
- net Out: now also Q17.1 (D), R99.2
- net +3.3V renamed 3.3IN
- net In renamed Gate
- net Gate: now also R97.1
- new net: D49.2 (A), R97.2

Commit message: pedning review
Parts:
- C64: value 100nF -> 100n
- R98: value 100K -> 100k
- R99: value 10K -> 10k
Changed lines of the file:
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@@
 			)
 		)
-		(property "Value" "100nF"
+		(property "Value" "100n"
 			(at 137.16 81.2799 0)
 			(show_name no)
@@
 			)
 		)
-		(property "Value" "10K"
+		(property "Value" "10k"
 			(at 153.67 60.9599 0)
 			(show_name no)
@@
 			)
 		)
-		(property "Value" "100K"
+		(property "Value" "100k"
 			(at 127 81.2799 0)
 			(show_name no)

Commit message: footprint! mising 2
Parts:
- C23: renamed from C64; footprint (none) -> Capacitor_SMD:C_0603_1608Metric_Pad1.08x0.95mm_HandSolder
- D19: renamed from D49; footprint (none) -> LED_SMD:LED_0603_1608Metric_Pad1.05x0.95mm_HandSolder
- Q4: renamed from Q17; footprint (none) -> LSOM_IRLM:SOT23; p/n (none) -> IRLML0030TRPBF
- R31: renamed from R97; footprint (none) -> Resistor_SMD:R_0603_1608Metric_Pad0.98x0.95mm_HandSolder
- R32: renamed from R98; footprint (none) -> Resistor_SMD:R_0603_1608Metric_Pad0.98x0.95mm_HandSolder
- R33: renamed from R99; footprint (none) -> Resistor_SMD:R_0603_1608Metric_Pad0.98x0.95mm_HandSolder
