File: hardware/ESP32.kicad_sch (KiCad schematic)
At the start: 21 parts, among them J3 USB_C_Receptacle_USB2.0_16P, SW2 BOOT Switch, SW3 RESET Button, U2 ESP32-C6-MINI-1

Commit message: organized
Parts:
- renumbered C15 to C13, C16 to C14, C17 to C15, C18 to C16, J3 to J1, R12 to R10, R13 to R11, R14 to R12, R15 to R13, R16 to R14, R9 to R7, R10 to R8, R11 to R9, SW2 to SW1, SW3 to SW2, U2 to U1
