File: hardware/ESP.kicad_sch (KiCad schematic)
At the start: 3 parts

Commit message: techuri
Connections:
- no-connect marks 0 -> 4
Other:
- moved on the sheet: R17
Changed lines of the file:
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@@
 	(generator_version "10.0")
 	(paper "A4")
-	(wire
-		(pts
-			(xy 207.01 88.9) (xy 214.63 88.9)
-		)
-		(stroke
-			(width 0)
-			(type default)
-		)
-	)
-	(wire
-		(pts
-			(xy 210.82 86.36) (xy 214.63 86.36)
+	(no_connect
+		(at 114.3 78.74)
+	)
+	(no_connect
+		(at 114.3 81.28)
+	)
+	(no_connect
+		(at 144.78 77.47)
+	)
+	(no_connect
+		(at 144.78 74.93)
+	)
+	(wire
+		(pts
+			(xy 205.74 93.98) (xy 213.36 93.98)
+		)
+		(stroke
+			(width 0)
+			(type default)
+		)
+	)
+	(wire
+		(pts
+			(xy 201.93 88.9) (xy 205.74 88.9)
 		)
 		(stroke
@@
 	(wire
 		(pts
-			(xy 210.82 83.82) (xy 214.63 83.82)
+			(xy 201.93 86.36) (xy 205.74 86.36)
 		)
 		(stroke
@@
 	(wire
 		(pts
-			(xy 194.31 88.9) (xy 199.39 88.9)
+			(xy 193.04 93.98) (xy 198.12 93.98)
 		)
 		(stroke
@@
 	)
 	(label "ESP_RESET"
-		(at 194.31 88.9 180)
+		(at 193.04 93.98 180)
 		(effects
 			(font
@@
 	)
 	(label "ESP_GPIO1"
-		(at 210.82 83.82 0)
-		(effects
-			(font
-				(size 1.27 1.27)
-			)
-			(justify left bottom)
+		(at 201.93 86.36 180)
+		(effects
+			(font
+				(size 1.27 1.27)
+			)
+			(justify right bottom)
 		)
 	)
@@
 	)
 	(label "ESP_GPIO2"
-		(at 210.82 86.36 0)
-		(effects
-			(font
-				(size 1.27 1.27)
-			)
-			(justify left bottom)
+		(at 201.93 88.9 180)
+		(effects
+			(font
+				(size 1.27 1.27)
+			)
+			(justify right bottom)
 		)
 	)
@@
 	(hierarchical_label "ESP_RESET"
 		(shape bidirectional)
-		(at 214.63 88.9 0)
+		(at 213.36 93.98 0)
 		(effects
 			(font
@@
 	(hierarchical_label "ESP_GPIO1"
 		(shape bidirectional)
-		(at 214.63 83.82 0)
+		(at 205.74 86.36 0)
 		(effects
 			(font
@@
 	(hierarchical_label "ESP_GPIO2"
 		(shape bidirectional)
-		(at 214.63 86.36 0)
+		(at 205.74 88.9 0)
 		(effects
 			(font
@@
 	(symbol
 		(lib_id "Device:R")
-		(at 203.2 88.9 90)
+		(at 201.93 93.98 90)
 		(unit 1)
 		(body_style 1)
@@
 		(dnp no)
 		(property "Reference" "R17"
-			(at 199.898 90.932 90)
+			(at 201.676 96.266 90)
 			(show_name no)
 			(do_not_autoplace no)
@@
 		)
 		(property "Value" "1k"
-			(at 203.962 90.932 90)
+			(at 202.438 94.234 90)
 			(show_name no)
 			(do_not_autoplace no)
@@
 		)
 		(property "Footprint" ""
-			(at 203.2 90.678 90)
+			(at 201.93 95.758 90)
 			(hide yes)
 			(show_name no)
@@
 		)
 		(property "Datasheet" ""
-			(at 203.2 88.9 0)
+			(at 201.93 93.98 0)
 			(hide yes)
 			(show_name no)
@@
 		)
 		(property "Description" "Resistor"
-			(at 203.2 88.9 0)
+			(at 201.93 93.98 0)
 			(hide yes)
 			(show_name no)
@@
 		(dnp no)
 		(property "Reference" "R16"
-			(at 199.898 83.312 90)
+			(at 203.2 83.312 90)
 			(show_name no)
 			(do_not_autoplace no)
@@
 		)
 		(property "Value" "1k"
-			(at 203.962 83.312 90)
+			(at 203.708 81.28 90)
 			(show_name no)
 			(do_not_autoplace no)
@@
 		)
 		(property "Value" "1k"
-			(at 202.438 73.66 90)
-			(show_name no)
-			(do_not_autoplace no)
+			(at 202.946 78.74 90)
+			(show_name no)
+			(do_not_autoplace no)
