File: hardware/MCU.kicad_sch (KiCad schematic)
At the start: 4 parts, among them J1 Horn Plug in, J7 Steering Wheel, J9 Dashboard IO, Q15 NMOS

Commit message: sahty
Other:
- added sheet CANS (CANS.kicad_sch)
Changed lines of the file:
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@@
+	)
+	(sheet
+		(at 36.83 154.94)
+		(size 30.48 24.13)
+		(exclude_from_sim no)
+		(in_bom yes)
+		(on_board yes)
+		(dnp no)
+		(fields_autoplaced yes)
+		(stroke
+			(width 0.1524)
+			(type solid)
+		)
+		(fill
+			(color 0 0 0 0)
+		)
+		(property "Sheetname" "CANS"
+			(at 36.83 154.2284 0)
+			(show_name no)
+			(do_not_autoplace no)
+			(effects
+				(font
+					(size 1.27 1.27)
+				)
+				(justify left bottom)
+			)
+		)
+		(property "Sheetfile" "CANS.kicad_sch"
+			(at 36.83 179.6546 0)
+			(show_name no)
+			(do_not_autoplace no)
+			(effects
+				(font
+					(size 1.27 1.27)
+				)
+				(justify left top)
+			)
+		)
+		(instances
+			(project "DEI"
+				(path "/1469f349-54e5-4a37-953e-ac48c70e29b2/2751c2d7-629c-4bb6-8dd2-1a829c053e6c"
+					(page "2")
+				)
+			)
+		)
 	)
 	(sheet

Commit message: oh shittings
Parts:
- added J10, J12, J8: Steering_Can_Out, symbol Connector_Generic:Conn_01x02
Connections:
- new net Car_Can/CAN_H: J12.1 (Pin_1)
- new net Car_Can/CAN_L: J12.2 (Pin_2)
- new net Lighting_Can/CAN_H: J10.1 (Pin_1)
- new net Lighting_Can/CAN_L: J10.2 (Pin_2)
- new net Steering_Can/CAN_H: J8.1 (Pin_1)
- new net Steering_Can/CAN_L: J8.2 (Pin_2)
Other:
- removed sheet CANS
- added sheet Car_Can (test.kicad_sch)
- added sheet Lighting_Can (test.kicad_sch)
- added sheet Lights (Lights.kicad_sch)
- added sheet Steering_Can (test.kicad_sch)

Commit message: meow
Parts:
- removed J1: Horn Plug in, symbol Connector_Generic:Conn_01x02
Connections:
- net Horn Plug In: now reaches Q15.3 (S)
Changed lines of the file:
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@@
 	(generator_version "10.0")
 	(paper "A4")
+	(rectangle
+		(start 200.66 132.08)
+		(end 200.66 132.08)
+		(stroke
+			(width 0)
+			(type default)
+		)
+		(fill
+			(type none)
+		)
+	)
+	(rectangle
+		(start 15.24 144.78)
+		(end 142.24 185.42)
+		(stroke
+			(width 0)
+			(type default)
+		)
+		(fill
+			(type none)
+		)
+	)
+	(rectangle
+		(start 157.48 15.24)
+		(end 157.48 15.24)
+		(stroke
+			(width 0)
+			(type default)
+		)
+		(fill
+			(type none)
+		)
+	)
+	(rectangle
+		(start 25.4 81.28)
+		(end 27.94 83.82)
+		(stroke
+			(width 0)
+			(type default)
+		)
+		(fill
+			(type none)
+		)
+	)
+	(rectangle
+		(start 165.1 15.24)
+		(end 190.5 127)
+		(stroke
+			(width 0)
+			(type default)
+		)
+		(fill
+			(type none)
+		)
+	)
+	(rectangle
+		(start 25.4 86.36)
+		(end 66.04 116.84)
+		(stroke
+			(width 0)
+			(type default)
+		)
+		(fill
+			(type none)
+		)
+	)
 	(junction
 		(at 153.67 83.82)
@@
 	(wire
 		(pts
-			(xy 168.91 120.65) (xy 156.21 120.65)
+			(xy 50.8 95.25) (xy 59.69 95.25)
 		)
 		(stroke
@@
 	(wire
 		(pts
-			(xy 81.28 95.25) (xy 85.09 95.25)
+			(xy 168.91 120.65) (xy 156.21 120.65)
 		)
 		(stroke
@@
 	(wire
 		(pts
-			(xy 153.67 83.82) (xy 186.69 83.82)
+			(xy 81.28 95.25) (xy 85.09 95.25)
 		)
 		(stroke
@@
 	(wire
 		(pts
-			(xy 213.36 66.04) (xy 219.71 66.04)
+			(xy 153.67 83.82) (xy 186.69 83.82)
 		)
 		(stroke
@@
 	(wire
 		(pts
-			(xy 43.18 92.71) (xy 43.18 95.25)
+			(xy 213.36 66.04) (xy 219.71 66.04)
 		)
 		(stroke
@@
 	(wire
 		(pts
-			(xy 43.18 95.25) (xy 59.69 95.25)
-		)
-		(stroke
-			(width 0)
-			(type default)
-		)
-	)
-	(wire
-		(pts
 			(xy 166.37 82.55) (xy 167.64 82.55)
 		)
@@
 	(wire
 		(pts
-			(xy 35.56 90.17) (xy 43.18 90.17)
-		)
-		(stroke
-			(width 0)
-			(type default)
-		)
-	)
-	(wire
-		(pts
 			(xy 153.67 116.84) (xy 190.5 116.84)
 		)
@@
 		)
 	)
-	(hierarchical_label "12V"
-		(shape input)
-		(at 35.56 90.17 180)
-		(effects
-			(font
-				(size 1.27 1.27)
-			)
-			(justify right)
-		)
-	)
 	(hierarchical_label "ESP_UART_TX"
 		(shape output)
@@
 		)
 	)
+	(hierarchical_label "Horn Plug In"
+		(shape output)
+		(at 50.8 95.25 180)
+		(effects
+			(font
+				(size 1.27 1.27)
+			)
+			(justify right)
+		)
+	)
 	(hierarchical_label "ESP_UART_RX"
 		(shape output)
@@
 					(unit 1)
 				)
-			)
-		)
-	)
-	(symbol
-		(lib_id "Connector_Generic:Conn_01x02")
-		(at 48.26 90.17 0)
-		(unit 1)
-		(body_style 1)
-		(exclude_from_sim no)
-		(in_bom yes)
-		(on_board yes)
-		(in_pos_files yes)
-		(dnp no)
-		(fields_autoplaced yes)
-		(property "Reference" "J1"
-			(at 50.8 90.1699 0)
-			(show_name no)
-			(do_not_autoplace no)
-			(effects
-				(font
-					(size 1.27 1.27)
-				)
-				(justify left)
-			)
-		)
-		(property "Value" "Horn Plug in"
-			(at 50.8 92.7099 0)
-			(show_name no)
-			(do_not_autoplace no)
-			(effects
-				(font
-					(size 1.27 1.27)
-				)
-				(justify left)
-			)
-		)
-		(property "Footprint" ""
-			(at 48.26 90.17 0)
-			(hide yes)
-			(show_name no)
-			(do_not_autoplace no)
-			(effects
-				(font
-					(size 1.27 1.27)
-				)
-			)
-		)
-		(property "Datasheet" ""
-			(at 48.26 90.17 0)
-			(hide yes)
-			(show_name no)
-			(do_not_autoplace no)
-			(effects
-				(font
-					(size 1.27 1.27)
-				)
-			)
-		)
-		(property "Description" "Generic connector, single row, 01x02, script generated (kicad-library-utils/schlib/autogen/connector/)"
-			(at 48.26 90.17 0)
-			(hide yes)
-			(show_name no)
-			(do_not_autoplace no)
-			(effects
-				(font
-					(size 1.27 1.27)
-				)
-			)
-		)
-		(pin "1"
-		)
-		(pin "2"
-		)
-		(instances
-			(project "DEI"
-				(path "/1469f349-54e5-4a37-953e-ac48c70e29b2/2751c2d7-629c-4bb6-8dd2-1a829c053e6c"
-					(reference "J1")
-					(unit 1)
-				)

Commit message: organized
Parts:
- removed J10, J12, J8: Steering_Can_Out, symbol Connector_Generic:Conn_01x02
- removed J7: Steering Wheel, symbol Connector_Generic:Conn_01x04
- removed J9: Dashboard IO, symbol Connector_Generic:Conn_02x05_Odd_Even
- added C17: 100nf, symbol Device:C
- added R69: 1k, symbol Device:R
- added R70: 10K, symbol Device:R
Connections:
- net 100PinMCU/NRST: now also C17.1, R69.2
- net ESP_GPIO1: now also R69.1
- net ESP_GPIO2: now also R70.1
- net GND: now also C17.2, R70.2
Other:
- sheet 100PinMCU ports: added none; removed GNDA

Commit message: techuri
Connections:
- no-connect marks 0 -> 56
Other:
- note added: "Dashboard and Sgteering wheel Inputs"
- note added: "FET protection"
- moved on the sheet: R70

Commit message: eja
Parts:
- added D15, D16, D17: Status LED, symbol Device:LED
- added R72, R74, R75: 1k, symbol Device:R
Connections:
- net 100PinMCU/PF10: now also R75.2
- net 100PinMCU/PF2: now also R74.2
- net 100PinMCU/PF9: now also R72.2
- net GND: now also D15.1 (K), D16.1 (K), D17.1 (K)
- new net: D17.2 (A), R75.1
- new net: D15.2 (A), R72.1
- new net: D16.2 (A), R74.1
- no-connect marks 56 -> 53
Other:
- removed sheet Car_Can
- removed sheet Lighting_Can
- removed sheet Steering_Can
- added sheet CAN_Transceiver (CAN_Transceiver.kicad_sch)
- added sheet Car_Transceiver (CAN_Transceiver.kicad_sch)
- added sheet Lighting_Transceiver (CAN_Transceiver.kicad_sch)

Commit message: someone please check if i fucked up removing boot
Parts:
- removed C17: 100nf, symbol Device:C
- removed D15, D16, D17: Status LED, symbol Device:LED
- removed Q15: NMOS, symbol Simulation_SPICE:NMOS
- removed R69, R72, R74, R75: 1k, symbol Device:R
- added C74: 100nf, symbol Device:C
- added D21, D22, D31: Status LED, symbol Device:LED
- added R76, R77, R78: 1k, symbol Device:R
- added R79: 2.2k, symbol Device:R
Connections:
- net ESP_GPIO1: now also R76.1
- net GND: now also C74.2, D21.1 (K), D22.1 (K), D31.1 (K)
- new net: D31.2 (A), R79.2
- new net: D22.2 (A), R78.1
- new net: D21.2 (A), R77.1
- new net 48PinMCU/NRST: C74.1, R76.2
- new net 48PinMCU/PB12: R78.2
- new net 48PinMCU/PB13: R77.2
- new net USB5V: R79.1
- no-connect marks 53 -> 6
Other:
- removed sheet 100PinMCU
- added sheet 48PinMCU (48PinMCU.kicad_sch)
- added sheet USB-C_Connector (USB-C_Connector.kicad_sch)
- note removed: "Dashboard and Sgteering wheel Inputs"
- moved on the sheet: R70

Commit message: ready for round 3
Parts:
- removed R70: 10K, symbol Device:R
- removed R76: 1k, symbol Device:R
- added SW10, SW4, SW6, SW7, SW8, SW9: SW_Push, symbol Switch:SW_Push
Connections:
- net +3.3V: now also SW10.1, SW4.1, SW6.1, SW7.1, SW8.1, SW9.1
- net GEAR_F_IN: now also SW7.2
- net GEAR_R_IN: now also SW8.2
- net IGN_ARR_IN: now also SW4.2
- net IGN_MTR_IN: now also SW6.2
- net Turn_L_IN: now also SW10.2
- net Turn_R_IN: now also SW9.2
Other:
- removed sheet NMOS8
- note added: "Dashboard Input Fet"
- note added: "Steering Wheel Fet"
- note removed: "FET protection"
