File: hardware/MCU.kicad_sch (KiCad schematic)
At the start: 13 parts, among them SW10 SW_Push, SW4 SW_Push, SW6 SW_Push, SW7 SW_Push, SW8 SW_Push, SW9 SW_Push

Commit message: rawr
Parts:
- removed C74: 100nf, symbol Device:C
- removed D21, D22, D31: Status LED, symbol Device:LED
- removed R77, R78: 1k, symbol Device:R
- removed R79: 2.2k, symbol Device:R
- removed SW10, SW4, SW6, SW7, SW8, SW9: SW_Push, symbol Switch:SW_Push
- added C75: 100nf, symbol Device:C
- added D36, D37: Status LED, symbol Device:LED
- added R83, R84: 1k, symbol Device:R
- added SW2, SW4, SW6: SW_SP3T_NR01103, Button_Switch_THT:SW_NKK_NR01, symbol Switch:SW_SP3T_NR01103
Connections:
- net GEAR_F_IN: now also SW4.1
- net GEAR_R_IN: now also SW4.3
- net GND: now also C75.2, D36.1 (K), D37.1 (K)
- net IGN_ARR_IN: now also SW2.2
- net IGN_MTR_IN: now also SW2.1
- net Turn_L_IN: now also SW6.1
- net Turn_R_IN: now also SW6.3
- new net: D36.2 (A), R83.1
- new net: D37.2 (A), R84.1
- new net 100PinMCU/NRST: C75.1
- new net 100PinMCU/PB12: R83.2
- new net 100PinMCU/PB13: R84.2
- new net 3.3IN: SW2.C (Common), SW4.C (Common), SW6.C (Common)
- new net Gear_N: SW4.2
- new net IGN_Off: SW2.3
- new net Steering_M: SW6.2
- no-connect marks 6 -> 50
Other:
- removed sheet 48PinMCU
- removed sheet Lighting_Transceiver
- removed sheet Lights
- removed sheet NMOS
- removed sheet NMOS1
- removed sheet NMOS10
- removed sheet NMOS2
- removed sheet NMOS9
- removed sheet USB-C_Connector
- added sheet 100PinMCU (100PinMCU.kicad_sch)
- added sheet Llighting_trans (CAN_Transceiver.kicad_sch)
- added sheet NMOS12 (NMOS.kicad_sch)
- added sheet NMOS13 (NMOS.kicad_sch)
- added sheet NMOS14 (NMOS.kicad_sch)
- added sheet NMOS15 (NMOS.kicad_sch)
- added sheet NMOS16 (NMOS.kicad_sch)
- added sheet NMOS17 (NMOS.kicad_sch)
- added sheet NMOS18 (NMOS.kicad_sch)
- added sheet NMOS19 (NMOS.kicad_sch)
- sheet NMOS11 ports: added 3.3IN, Gate; removed In
- sheet NMOS3 ports: added 3.3IN, Gate; removed In
- sheet NMOS4 ports: added 3.3IN, Gate; removed In
- sheet NMOS5 ports: added 3.3IN, Gate; removed In
- sheet NMOS6 ports: added 3.3IN, Gate; removed In
- sheet NMOS7 ports: added 3.3IN, Gate; removed In

Commit message: pedning review
Parts:
- added D38, D45, D47, D56, D57: Status LED, symbol Device:LED
- added D44: Status LEDs, symbol Device:LED
- added R116, R117, R88, R89, R92, R93: 1k, symbol Device:R
- C75: value 100nf -> 100n
- SW2, SW4, SW6: now fitted
Connections:
- net 100PinMCU/PE6: now also R116.2
- net 100PinMCU/PE7: now also R117.2
- net 100PinMCU/PE8: now also R92.2
- net 100PinMCU/PE9: now also R93.2
- net 100PinMCU/PF10: now also R88.2
- net 100PinMCU/PF2: now also R89.2
- net GND: now also D38.1 (K), D44.1 (K), D45.1 (K), D47.1 (K), D56.1 (K), D57.1 (K)
- new net: D47.2 (A), R117.1
- new net: D44.2 (A), R89.1
- new net: D45.2 (A), R93.1
- new net: D57.2 (A), R116.1
- new net: D56.2 (A), R92.1
- new net: D38.2 (A), R88.1
- no-connect marks 50 -> 44

Commit message: footprint! mising 2
Parts:
- added SW5: Regen, Button_Switch_THT:SW_PUSH_6mm, symbol Switch:SW_Push
- added SW6: Cruise, Button_Switch_THT:SW_PUSH_6mm, symbol Switch:SW_Push
- added SW7: Cruise Enable, Button_Switch_THT:SW_PUSH_6mm, symbol Switch:SW_Push
- added SW8: Hazard, Button_Switch_THT:SW_PUSH_6mm, symbol Switch:SW_Push
- added SW9: Horn, Button_Switch_THT:SW_PUSH_6mm, symbol Switch:SW_Push
- C22: renamed from C75; footprint (none) -> Capacitor_SMD:C_0603_1608Metric_Pad1.08x0.95mm_HandSolder
- D11: renamed from D57; footprint (none) -> LED_SMD:LED_0603_1608Metric_Pad1.05x0.95mm_HandSolder
- D12: renamed from D47; footprint (none) -> LED_SMD:LED_0603_1608Metric_Pad1.05x0.95mm_HandSolder
- D13: renamed from D56; footprint (none) -> LED_SMD:LED_0603_1608Metric_Pad1.05x0.95mm_HandSolder
- D14: renamed from D45; footprint (none) -> LED_SMD:LED_0603_1608Metric_Pad1.05x0.95mm_HandSolder
- D15: renamed from D38; footprint (none) -> LED_SMD:LED_0603_1608Metric_Pad1.05x0.95mm_HandSolder
- D16: renamed from D44; value Status LEDs -> Firmware- Green LEDs; footprint (none) -> LED_SMD:LED_0603_1608Metric_Pad1.05x0.95mm_HandSolder
- D17: renamed from D36; footprint (none) -> LED_SMD:LED_0603_1608Metric_Pad1.05x0.95mm_HandSolder
- D18: renamed from D37; value Status LED -> Firmware green led; footprint (none) -> LED_SMD:LED_0603_1608Metric_Pad1.05x0.95mm_HandSolder
- R23: renamed from R116; footprint (none) -> Resistor_SMD:R_0603_1608Metric_Pad0.98x0.95mm_HandSolder
- R24: renamed from R117; footprint (none) -> Resistor_SMD:R_0603_1608Metric_Pad0.98x0.95mm_HandSolder
- R25: renamed from R92; footprint (none) -> Resistor_SMD:R_0603_1608Metric_Pad0.98x0.95mm_HandSolder
- R26: renamed from R93; footprint (none) -> Resistor_SMD:R_0603_1608Metric_Pad0.98x0.95mm_HandSolder
- R27: renamed from R88; footprint (none) -> Resistor_SMD:R_0603_1608Metric_Pad0.98x0.95mm_HandSolder
- R28: renamed from R89; footprint (none) -> Resistor_SMD:R_0603_1608Metric_Pad0.98x0.95mm_HandSolder
- R29: renamed from R83; footprint (none) -> Resistor_SMD:R_0603_1608Metric_Pad0.98x0.95mm_HandSolder
- R30: renamed from R84; footprint (none) -> Resistor_SMD:R_0603_1608Metric_Pad0.98x0.95mm_HandSolder
- renumbered SW2 to SW1, SW4 to SW2, SW6 to SW3
Connections:
- net 3.3IN: now also SW5.2, SW6.2, SW7.2, SW8.2, SW9.2
- net GEAR_R_IN renamed NMOS16/Gate
- new net NMOS11/Gate: SW9.1
- new net NMOS4/Gate: SW7.1
- new net NMOS5/Gate: SW6.1
- new net NMOS6/Gate: SW5.1
- new net NMOS7/Gate: SW8.1
Other:
- note added: "TIM3_CH1"
- note added: "TIM3_CH2"
- note added: "TIM3_CH3"
- note added: "TIM4_CH1"
- note added: "TIM4_CH2"
- note added: "TIM4_CH3"
