File: hardware/DEI.kicad_sch (KiCad schematic)
At the start: 35 parts, among them J1 Supp_In, J10 Steering_Can, J12 Car_Can, J13 Steering_Can, J15 Horn, J16 Supp_out, J17 ESTOP Connector, J18 ESTOP IN, J19 LLS, J20 RLS, J21 Steering_Can_Debug, J22 Lighting_Can_Debug, J23 Car_Can_Debug, J24 HeadLight_Left, J25 HeadLight_Right, J26 Lighting_Can, J27 Lighting_Can, J4 Power Input, J6 Car_Can, J8 Dashboard, J9 Steering Wheel, Q15 NMOS

Commit message: pedning review
Parts:
- C13: value 100uf -> 100u
Connections:
- net 12V_PP is gone; now on net 12V_Light: J26.1 (12V), J27.1 (12V)
Other:
- sheet MCU ports: added USB_D+, USB_D-; removed ESP_RESET, USB_DM, USB_DP
- sheet Power ports: added none; removed 12V_PP
- moved on the sheet: J12, J21, J22, J23, J6, R34, R67
