File: hardware/DEI.kicad_sch (KiCad schematic)
At the start: 35 parts, among them J1 Supp_In, J10 Steering_Can, J12 Car_Can, J13 Steering_Can, J15 Horn, J16 Supp_out, J17 ESTOP Connector, J18 ESTOP IN, J19 LLS, J20 RLS, J21 Steering_Can_Debug, J22 Lighting_Can_Debug, J23 Car_Can_Debug, J24 HeadLight_Left, J25 HeadLight_Right, J26 Lighting_Can, J27 Lighting_Can, J4 Power Input, J6 Car_Can, J8 Dashboard, J9 Steering Wheel, Q15 NMOS

Commit message: sahtyyyyy
Parts:
- D4: value D -> D - VSSAF510HM3/H
Other:
- note added: "ESTOP"
- moved on the sheet: C13, D31, D4, H1, H2, H3, H4, J10, J13, J15, J4, J8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
