File: hardware/DEI.kicad_sch (KiCad schematic)
At the start: 35 parts, among them J1 Supp_In, J10 Steering_Can, J12 Car_Can, J13 Steering_Can, J15 Horn, J16 Supp_out, J17 ESTOP Connector, J18 ESTOP IN, J19 LLS, J20 RLS, J21 Steering_Can_Debug, J22 Lighting_Can_Debug, J23 Car_Can_Debug, J24 HeadLight_Left, J25 HeadLight_Right, J26 Lighting_Can, J27 Lighting_Can, J4 Power Input, J6 Car_Can, J8 Dashboard, J9 Steering Wheel, Q15 NMOS

Commit message: footprint! mising 2
Parts:
- removed J8: Dashboard, symbol Connector_Generic:Conn_02x06_Odd_Even
- removed J9: Steering Wheel, symbol Connector_Generic:Conn_01x05
- C1: renamed from C13; footprint (none) -> Capacitor_SMD:C_0603_1608Metric_Pad1.08x0.95mm_HandSolder
- D1: renamed from D4; value D - VSSAF510HM3/H -> D
- D2: renamed from D31; footprint (none) -> LED_SMD:LED_0603_1608Metric_Pad1.05x0.95mm_HandSolder
- J1: footprint (none) -> LHRS_Connectors:AMASS_XT30UPB-M_1x02_P5.0mm_Vertical
- J13: renamed from J17; footprint (none) -> LHRS_Connectors:Molex_Nano-Fit_105309-xx04_1x04_P2.50mm_Vertical
- J16: renamed from J19; footprint (none) -> LHRS_Connectors:Molex_Nano-Fit_105309-xx04_1x04_P2.50mm_Vertical
- J17: renamed from J20; footprint (none) -> LHRS_Connectors:Molex_Nano-Fit_105309-xx04_1x04_P2.50mm_Vertical
- J19: renamed from J24; footprint (none) -> LHRS_Connectors:Molex_Nano-Fit_105309-xx04_1x04_P2.50mm_Vertical
- J2: renamed from J16; footprint (none) -> LHRS_Connectors:AMASS_XT30UPB-M_1x02_P5.0mm_Vertical
- J20: renamed from J25; footprint (none) -> LHRS_Connectors:Molex_Nano-Fit_105309-xx04_1x04_P2.50mm_Vertical
- J21: renamed from J15; footprint (none) -> LHRS_Connectors:AMASS_XT30UPB-M_1x02_P5.0mm_Vertical
- J3: renamed from J4; footprint (none) -> LHRS_Connectors:MX150_02x02_Vertical
- J8: renamed from J18; footprint (none) -> LHRS_Connectors:AMASS_XT30UPB-M_1x02_P5.0mm_Vertical
- Q1: renamed from Q15; footprint (none) -> LSOM_IRLM:SOT23; p/n (none) -> IRLML0030TRPBF
- R1: renamed from R34; footprint (none) -> Resistor_SMD:R_0603_1608Metric_Pad0.98x0.95mm_HandSolder
- R2: renamed from R1; footprint (none) -> Resistor_SMD:R_0603_1608Metric_Pad0.98x0.95mm_HandSolder
- R3: renamed from R67; footprint (none) -> Resistor_SMD:R_0603_1608Metric_Pad0.98x0.95mm_HandSolder
- R4: renamed from R2; footprint (none) -> Resistor_SMD:R_0603_1608Metric_Pad0.98x0.95mm_HandSolder
- R5: renamed from R7; footprint (none) -> Resistor_SMD:R_0603_1608Metric_Pad0.98x0.95mm_HandSolder
- R6: renamed from R79; footprint (none) -> Resistor_SMD:R_0603_1608Metric_Pad0.98x0.95mm_HandSolder
- renumbered H3 to H2, H2 to H3, J27 to J10, J10 to J11, J21 to J12, J13 to J15, J6 to J4, J23 to J5, J26 to J6, J12 to J7, J22 to J9
Connections:
- no-connect marks 1 -> 2
Other:
- sheet MCU ports: added none; removed CRUISE_EN_IN, CRUISE_SET_IN, GEAR_F_IN, GEAR_R_IN, Gear_N, HAZARD_IN, Horn_IN, IGN_ARR_IN, IGN_MTR_IN, IGN_Off, REGEN_EN_IN, Steering_M, Turn_L_IN, Turn_R_IN
- sheet USB-C_Connector ports: added CC1, CC2; removed none
- note removed: "Steering and Dashboard IO"
- moved on the sheet: D2, J13, J16, J17, J19, J20, R6
