File: hardware/100PinMCU.kicad_sch (KiCad schematic)
At the start: 33 parts, among them J1 SWD_Header, J2 SWD, SW1 SW_SPDT, U1 STM32G473VETx, Y1 Crystal

Commit message: mcu and power
Parts:
- renumbered C1 to C34, C2 to C35, C3 to C36, C4 to C37, C5 to C38, C6 to C39, C7 to C40, C8 to C41, C9 to C42, C10 to C43, C11 to C44, C12 to C45, C13 to C46, C14 to C47, D1 to D12, D2 to D13, D3 to D14, FB1 to FB3, FB2 to FB4, J1 to J5, J2 to J6, R1 to R25, R2 to R26, R3 to R27, R4 to R28, R5 to R29, R6 to R30, R7 to R31, R8 to R32, Reset1 to Reset2, SW1 to SW4, U1 to U5, Y1 to Y2

Commit message: rawr
Parts:
- removed C36: 10u, Capacitor_SMD:C_0805_2012Metric, symbol Device:C
- removed C37, C38, C39, C40, C41, C43, C45, C46: 0.1u, Capacitor_SMD:C_0603_1608Metric_Pad1.08x0.95mm_HandSolder, symbol Device:C
- removed C42, C44: 1u, Capacitor_SMD:C_0603_1608Metric_Pad1.08x0.95mm_HandSolder, symbol Device:C
- removed R25: 10k, Resistor_SMD:R_0603_1608Metric_Pad0.98x0.95mm_HandSolder, symbol Device:R
- removed Reset2: Reset, LHRS_Special:TL3365AF180QG, symbol Switch:SW_Push
- added C81: 10u, Capacitor_SMD:C_0805_2012Metric, symbol Device:C
- added C82, C83, C84, C85, C86, C88, C90, C91: 0.1u, Capacitor_SMD:C_0603_1608Metric_Pad1.08x0.95mm_HandSolder, symbol Device:C
- added C87, C89: 1u, Capacitor_SMD:C_0603_1608Metric_Pad1.08x0.95mm_HandSolder, symbol Device:C
- added R52: 10k, Resistor_SMD:R_0603_1608Metric_Pad0.98x0.95mm_HandSolder, symbol Device:R
- added Reset1: Reset, LHRS_Special:TL3365AF180QG, symbol Switch:SW_Push
- renumbered C34 to C79, C35 to C80, C47 to C92, D12 to D20, D13 to D27, D14 to D35, FB3 to FB5, FB4 to FB6, J5 to J28, J6 to J29, R26 to R55, R27 to R57, R28 to R58, R29 to R59, R30 to R71, R31 to R72, R32 to R73, SW4 to SW1, U5 to U6, Y2 to Y3
Connections:
- net +3V3: now also C81.1, C83.1, C86.1, C88.1, C90.1, C91.1, R52.2
- net GND: now also C81.2, C83.2, C85.2, C86.2, C88.2, C90.2, C91.2, Reset1.2
- net GNDA: now also C82.2, C84.2, C87.2, C89.2
- net NRST: now also C85.1, R52.1, Reset1.1
- net VDDA: now also C82.1, C84.1, C87.1, C89.1

Commit message: footprint! mising 2
Parts:
- renumbered C79 to C47, C80 to C48, C81 to C49, C82 to C50, C83 to C51, C84 to C52, C85 to C53, C86 to C54, C87 to C55, C88 to C56, C89 to C57, C90 to C58, C91 to C59, C92 to C60, D20 to D34, D27 to D35, D35 to D36, FB5 to FB1, FB6 to FB2, J28 to J23, J29 to J24, R52 to R72, R55 to R73, R57 to R74, R58 to R75, R59 to R76, R71 to R77, R72 to R78, R73 to R79, SW1 to SW4, U6 to U4, Y3 to Y1
