File: hardware/12VBuck.kicad_sch (KiCad schematic)
At the start: 14 parts, among them U3 LMR51635XDDCR

Commit message: techuri
Changed lines of the file:
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@@
+	(wire
+		(pts
+			(xy 0.0762 0.0762) (xy 12.7762 0.0762)
+		)
+		(stroke
+			(width 0)
+			(type default)
+		)
+	)
 	(wire
 		(pts

Commit message: someone please check if i fucked up removing boot
Parts:
- removed TP2: CB, TestPoint:TestPoint_THTPad_D3.0mm_Drill1.5mm, symbol Connector:TestPoint
- removed TP3: FB, TestPoint:TestPoint_THTPad_D3.0mm_Drill1.5mm, symbol Connector:TestPoint
- removed TP4: SW, TestPoint:TestPoint_THTPad_D3.0mm_Drill1.5mm, symbol Connector:TestPoint

Commit message: rawr
Parts:
- removed TP1: V_in_12V, TestPoint:TestPoint_THTPad_D3.0mm_Drill1.5mm, symbol Connector:TestPoint
- L1: footprint LHRS_Passives:74439369082 -> LHRS_Power:XAL5050822MEC; LCSC P/N (none) -> C5309356; P/N 74439369082 -> XAL5050-822MEC
- U1: renamed from U3; LCSC P/N (none) -> C42432812; P/N (none) -> LMR51635XDDCR
- renumbered C21 to C10, C22 to C11, C23 to C12, C24 to C15, C19 to C8, C20 to C9, R17 to R12, R18 to R13
Other:
- note added: "Vin: 4.6V to 60V"
- note removed: "Test Points"

Commit message: footprint! mising 2
Parts:
- renumbered C8 to C10, C9 to C11, C10 to C12, C11 to C13, C12 to C14, R12 to R15, R13 to R16
Changed lines of the file:
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@@
 		(dnp no)
 		(fields_autoplaced yes)
-		(property "Reference" "#FLG02"
+		(property "Reference" "#FLG03"
 			(at 149.86 79.375 0)
 			(hide yes)
@@
 			(project "DEI"
 				(path "/1469f349-54e5-4a37-953e-ac48c70e29b2/d41a835d-0002-40e6-b2c5-562251bf7d32/8dd4a490-1c92-4af5-a50b-9e0ac26eceaa"
-					(reference "#FLG02")
+					(reference "#FLG03")
 					(unit 1)
 				)
@@
 		(dnp no)
 		(fields_autoplaced yes)
-		(property "Reference" "C8"
+		(property "Reference" "C10"
 			(at 96.52 85.0962 0)
 			(show_name no)
@@
 			(project "DEI"
 				(path "/1469f349-54e5-4a37-953e-ac48c70e29b2/d41a835d-0002-40e6-b2c5-562251bf7d32/8dd4a490-1c92-4af5-a50b-9e0ac26eceaa"
-					(reference "C8")
+					(reference "C10")
 					(unit 1)
 				)
@@
 		(dnp no)
 		(fields_autoplaced yes)
-		(property "Reference" "#FLG04"
+		(property "Reference" "#FLG05"
 			(at 179.07 84.455 0)
 			(hide yes)
@@
 			(project "DEI"
 				(path "/1469f349-54e5-4a37-953e-ac48c70e29b2/d41a835d-0002-40e6-b2c5-562251bf7d32/8dd4a490-1c92-4af5-a50b-9e0ac26eceaa"
-					(reference "#FLG04")
+					(reference "#FLG05")
 					(unit 1)
 				)
@@
 		(dnp no)
 		(fields_autoplaced yes)
-		(property "Reference" "#FLG01"
+		(property "Reference" "#FLG02"
 			(at 88.9 79.375 0)
 			(hide yes)
@@
 			(project "DEI"
 				(path "/1469f349-54e5-4a37-953e-ac48c70e29b2/d41a835d-0002-40e6-b2c5-562251bf7d32/8dd4a490-1c92-4af5-a50b-9e0ac26eceaa"
-					(reference "#FLG01")
+					(reference "#FLG02")
 					(unit 1)
 				)
@@
 		(in_pos_files yes)
 		(dnp no)
-		(property "Reference" "C11"
+		(property "Reference" "C13"
 			(at 164.084 93.98 0)
 			(show_name no)
@@
 			(project "DEI"
 				(path "/1469f349-54e5-4a37-953e-ac48c70e29b2/d41a835d-0002-40e6-b2c5-562251bf7d32/8dd4a490-1c92-4af5-a50b-9e0ac26eceaa"
-					(reference "C11")
+					(reference "C13")
 					(unit 1)
 				)
@@
 		(in_pos_files yes)
 		(dnp no)
-		(property "Reference" "C10"
+		(property "Reference" "C12"
 			(at 156.718 80.01 0)
 			(show_name no)
@@
 			(project "DEI"
 				(path "/1469f349-54e5-4a37-953e-ac48c70e29b2/d41a835d-0002-40e6-b2c5-562251bf7d32/8dd4a490-1c92-4af5-a50b-9e0ac26eceaa"
-					(reference "C10")
+					(reference "C12")
 					(unit 1)
 				)
@@
 		(in_pos_files yes)
 		(dnp no)
-		(property "Reference" "#FLG03"
+		(property "Reference" "#FLG04"
 			(at 149.86 84.455 0)
 			(hide yes)
@@
 			(project "DEI"
 				(path "/1469f349-54e5-4a37-953e-ac48c70e29b2/d41a835d-0002-40e6-b2c5-562251bf7d32/8dd4a490-1c92-4af5-a50b-9e0ac26eceaa"
-					(reference "#FLG03")
+					(reference "#FLG04")
 					(unit 1)
 				)
@@
 		(dnp no)
 		(fields_autoplaced yes)
-		(property "Reference" "R12"
+		(property "Reference" "R15"
 			(at 227.33 85.0899 0)
 			(show_name no)
@@
 			(project "DEI"
 				(path "/1469f349-54e5-4a37-953e-ac48c70e29b2/d41a835d-0002-40e6-b2c5-562251bf7d32/8dd4a490-1c92-4af5-a50b-9e0ac26eceaa"
-					(reference "R12")
+					(reference "R15")
 					(unit 1)
 				)
@@
 		(dnp no)
 		(fields_autoplaced yes)
-		(property "Reference" "C9"
+		(property "Reference" "C11"
 			(at 105.41 87.6362 0)
 			(show_name no)
@@
 			(project "DEI"
 				(path "/1469f349-54e5-4a37-953e-ac48c70e29b2/d41a835d-0002-40e6-b2c5-562251bf7d32/8dd4a490-1c92-4af5-a50b-9e0ac26eceaa"
-					(reference "C9")
+					(reference "C11")
 					(unit 1)
 				)
@@
 		(dnp no)
 		(fields_autoplaced yes)
-		(property "Reference" "R13"
+		(property "Reference" "R16"
 			(at 227.33 92.7099 0)
 			(show_name no)
@@
 			(project "DEI"
 				(path "/1469f349-54e5-4a37-953e-ac48c70e29b2/d41a835d-0002-40e6-b2c5-562251bf7d32/8dd4a490-1c92-4af5-a50b-9e0ac26eceaa"
-					(reference "R13")
+					(reference "R16")
 					(unit 1)
 				)
@@
 		(in_pos_files yes)
 		(dnp no)
-		(property "Reference" "C12"
+		(property "Reference" "C14"
 			(at 173.482 94.234 0)
 			(show_name no)
@@
 			(project "DEI"
 				(path "/1469f349-54e5-4a37-953e-ac48c70e29b2/d41a835d-0002-40e6-b2c5-562251bf7d32/8dd4a490-1c92-4af5-a50b-9e0ac26eceaa"
-					(reference "C12")
-					(unit 1)
-				)
+					(reference "C14")
+					(unit 1)
+				)
