File: hardware/CAN_Transceiver.kicad_sch (KiCad schematic)
At the start: 9 parts, among them IC2 TCAN3413DR

Commit message: eja
Parts:
- renumbered C1 to C18, C2 to C60, C3 to C61, C4 to C62, D1 to D18, IC2 to IC5, JP1 to JP4, R1 to R43, R2 to R46

Commit message: rawr
Parts:
- renumbered C60 to C38, C61 to C39, C62 to C40, D18 to D10, IC5 to IC2, JP4 to JP2, R43 to R22, R46 to R23

Commit message: footprint! mising 2
Parts:
- renumbered C18 to C33, C38 to C34, C39 to C35, C40 to C36, D10 to D29, R22 to R61, R23 to R62
Changed lines of the file:
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@@
 		(in_pos_files yes)
 		(dnp no)
-		(property "Reference" "C38"
+		(property "Reference" "C34"
 			(at 76.2 73.66 0)
 			(show_name no)
@@
 			(project "DEI"
 				(path "/1469f349-54e5-4a37-953e-ac48c70e29b2/2751c2d7-629c-4bb6-8dd2-1a829c053e6c/04396aca-93e1-400a-bc7c-fde1e6cca844"
-					(reference "C46")
+					(reference "C42")
 					(unit 1)
 				)
 				(path "/1469f349-54e5-4a37-953e-ac48c70e29b2/2751c2d7-629c-4bb6-8dd2-1a829c053e6c/5beee3ad-dd7b-48cc-8ccf-0b36fcf9786a"
+					(reference "C34")
+					(unit 1)
+				)
+				(path "/1469f349-54e5-4a37-953e-ac48c70e29b2/2751c2d7-629c-4bb6-8dd2-1a829c053e6c/e26fdb1b-0065-4bb9-9c82-052d7a56471c"
 					(reference "C38")
-					(unit 1)
-				)
-				(path "/1469f349-54e5-4a37-953e-ac48c70e29b2/2751c2d7-629c-4bb6-8dd2-1a829c053e6c/e26fdb1b-0065-4bb9-9c82-052d7a56471c"
-					(reference "C42")
 					(unit 1)
 				)
@@
 		(in_pos_files yes)
 		(dnp no)
-		(property "Reference" "C40"
+		(property "Reference" "C36"
 			(at 194.564 88.646 0)
 			(show_name no)
@@
 			(project "DEI"
 				(path "/1469f349-54e5-4a37-953e-ac48c70e29b2/2751c2d7-629c-4bb6-8dd2-1a829c053e6c/04396aca-93e1-400a-bc7c-fde1e6cca844"
-					(reference "C56")
+					(reference "C44")
 					(unit 1)
 				)
 				(path "/1469f349-54e5-4a37-953e-ac48c70e29b2/2751c2d7-629c-4bb6-8dd2-1a829c053e6c/5beee3ad-dd7b-48cc-8ccf-0b36fcf9786a"
+					(reference "C36")
+					(unit 1)
+				)
+				(path "/1469f349-54e5-4a37-953e-ac48c70e29b2/2751c2d7-629c-4bb6-8dd2-1a829c053e6c/e26fdb1b-0065-4bb9-9c82-052d7a56471c"
 					(reference "C40")
-					(unit 1)
-				)
-				(path "/1469f349-54e5-4a37-953e-ac48c70e29b2/2751c2d7-629c-4bb6-8dd2-1a829c053e6c/e26fdb1b-0065-4bb9-9c82-052d7a56471c"
-					(reference "C44")
 					(unit 1)
 				)
@@
 		(in_pos_files yes)
 		(dnp no)
-		(property "Reference" "C39"
+		(property "Reference" "C35"
 			(at 88.138 73.66 0)
 			(show_name no)
@@
 			(project "DEI"
 				(path "/1469f349-54e5-4a37-953e-ac48c70e29b2/2751c2d7-629c-4bb6-8dd2-1a829c053e6c/04396aca-93e1-400a-bc7c-fde1e6cca844"
-					(reference "C47")
+					(reference "C43")
 					(unit 1)
 				)
 				(path "/1469f349-54e5-4a37-953e-ac48c70e29b2/2751c2d7-629c-4bb6-8dd2-1a829c053e6c/5beee3ad-dd7b-48cc-8ccf-0b36fcf9786a"
+					(reference "C35")
+					(unit 1)
+				)
+				(path "/1469f349-54e5-4a37-953e-ac48c70e29b2/2751c2d7-629c-4bb6-8dd2-1a829c053e6c/e26fdb1b-0065-4bb9-9c82-052d7a56471c"
 					(reference "C39")
-					(unit 1)
-				)
-				(path "/1469f349-54e5-4a37-953e-ac48c70e29b2/2751c2d7-629c-4bb6-8dd2-1a829c053e6c/e26fdb1b-0065-4bb9-9c82-052d7a56471c"
-					(reference "C43")
 					(unit 1)
 				)
@@
 		(in_pos_files yes)
 		(dnp no)
-		(property "Reference" "C18"
+		(property "Reference" "C33"
 			(at 65.278 73.66 0)
 			(show_name no)
@@
 			(project "DEI"
 				(path "/1469f349-54e5-4a37-953e-ac48c70e29b2/2751c2d7-629c-4bb6-8dd2-1a829c053e6c/04396aca-93e1-400a-bc7c-fde1e6cca844"
-					(reference "C45")
+					(reference "C41")
 					(unit 1)
 				)
 				(path "/1469f349-54e5-4a37-953e-ac48c70e29b2/2751c2d7-629c-4bb6-8dd2-1a829c053e6c/5beee3ad-dd7b-48cc-8ccf-0b36fcf9786a"
-					(reference "C18")
+					(reference "C33")
 					(unit 1)
 				)
 				(path "/1469f349-54e5-4a37-953e-ac48c70e29b2/2751c2d7-629c-4bb6-8dd2-1a829c053e6c/e26fdb1b-0065-4bb9-9c82-052d7a56471c"
-					(reference "C41")
+					(reference "C37")
 					(unit 1)
 				)
@@
 		(in_pos_files yes)
 		(dnp no)
-		(property "Reference" "R23"
+		(property "Reference" "R62"
 			(at 201.93 80.01 90)
 			(show_name no)
@@
 			(project "DEI"
 				(path "/1469f349-54e5-4a37-953e-ac48c70e29b2/2751c2d7-629c-4bb6-8dd2-1a829c053e6c/04396aca-93e1-400a-bc7c-fde1e6cca844"
-					(reference "R27")
+					(reference "R66")
 					(unit 1)
 				)
 				(path "/1469f349-54e5-4a37-953e-ac48c70e29b2/2751c2d7-629c-4bb6-8dd2-1a829c053e6c/5beee3ad-dd7b-48cc-8ccf-0b36fcf9786a"
-					(reference "R23")
+					(reference "R62")
 					(unit 1)
 				)
 				(path "/1469f349-54e5-4a37-953e-ac48c70e29b2/2751c2d7-629c-4bb6-8dd2-1a829c053e6c/e26fdb1b-0065-4bb9-9c82-052d7a56471c"
-					(reference "R25")
+					(reference "R64")
 					(unit 1)
 				)
@@
 		(dnp no)
 		(fields_autoplaced yes)
-		(property "Reference" "D10"
+		(property "Reference" "D29"
 			(at 196.85 46.99 0)
 			(show_name no)
@@
 			(project "DEI"
 				(path "/1469f349-54e5-4a37-953e-ac48c70e29b2/2751c2d7-629c-4bb6-8dd2-1a829c053e6c/04396aca-93e1-400a-bc7c-fde1e6cca844"
-					(reference "D12")
+					(reference "D31")
 					(unit 1)
 				)
 				(path "/1469f349-54e5-4a37-953e-ac48c70e29b2/2751c2d7-629c-4bb6-8dd2-1a829c053e6c/5beee3ad-dd7b-48cc-8ccf-0b36fcf9786a"
-					(reference "D10")
+					(reference "D29")
 					(unit 1)
 				)
 				(path "/1469f349-54e5-4a37-953e-ac48c70e29b2/2751c2d7-629c-4bb6-8dd2-1a829c053e6c/e26fdb1b-0065-4bb9-9c82-052d7a56471c"
-					(reference "D11")
+					(reference "D30")
 					(unit 1)
 				)
@@
 		(in_pos_files yes)
 		(dnp no)
-		(property "Reference" "R22"
+		(property "Reference" "R61"
 			(at 176.53 80.01 90)
 			(show_name no)
@@
 			(project "DEI"
 				(path "/1469f349-54e5-4a37-953e-ac48c70e29b2/2751c2d7-629c-4bb6-8dd2-1a829c053e6c/04396aca-93e1-400a-bc7c-fde1e6cca844"
-					(reference "R26")
+					(reference "R65")
 					(unit 1)
 				)
 				(path "/1469f349-54e5-4a37-953e-ac48c70e29b2/2751c2d7-629c-4bb6-8dd2-1a829c053e6c/5beee3ad-dd7b-48cc-8ccf-0b36fcf9786a"
-					(reference "R22")
+					(reference "R61")
 					(unit 1)
 				)
 				(path "/1469f349-54e5-4a37-953e-ac48c70e29b2/2751c2d7-629c-4bb6-8dd2-1a829c053e6c/e26fdb1b-0065-4bb9-9c82-052d7a56471c"
-					(reference "R24")
-					(unit 1)
-				)
+					(reference "R63")
+					(unit 1)
+				)
