File: hardware/Lights.kicad_sch (KiCad schematic)
At the start: 0 parts

Commit message: rawr
Other:
- added sheet Fetting_Head (Fetting.kicad_sch)
- added sheet Fetting_Left (Fetting.kicad_sch)
- added sheet Fetting_Right (Fetting.kicad_sch)

Commit message: pedning review
Changed lines of the file:
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@@
 	(wire
 		(pts
-			(xy 110.49 72.39) (xy 118.11 72.39)
-		)
-		(stroke
-			(width 0)
-			(type default)
-		)
-	)
-	(wire
-		(pts
-			(xy 82.55 45.72) (xy 88.9 45.72)
-		)
-		(stroke
-			(width 0)
-			(type default)
-		)
-	)
-	(wire
-		(pts
-			(xy 81.28 69.85) (xy 88.9 69.85)
-		)
-		(stroke
-			(width 0)
-			(type default)
-		)
-	)
-	(wire
-		(pts
-			(xy 110.49 60.96) (xy 118.11 60.96)
-		)
-		(stroke
-			(width 0)
-			(type default)
-		)
-	)
-	(wire
-		(pts
-			(xy 82.55 58.42) (xy 88.9 58.42)
+			(xy 88.9 69.85) (xy 82.55 69.85)
+		)
+		(stroke
+			(width 0)
+			(type default)
+		)
+	)
+	(wire
+		(pts
+			(xy 116.84 48.26) (xy 110.49 48.26)
+		)
+		(stroke
+			(width 0)
+			(type default)
+		)
+	)
+	(wire
+		(pts
+			(xy 118.11 72.39) (xy 110.49 72.39)
+		)
+		(stroke
+			(width 0)
+			(type default)
+		)
+	)
+	(wire
+		(pts
+			(xy 88.9 58.42) (xy 81.28 58.42)
+		)
+		(stroke
+			(width 0)
+			(type default)
+		)
+	)
+	(wire
+		(pts
+			(xy 116.84 60.96) (xy 110.49 60.96)
 		)
 		(stroke
@@
 	(wire
 		(pts
-			(xy 110.49 48.26) (xy 119.38 48.26)
+			(xy 88.9 44.45) (xy 80.01 44.45)
 		)
 		(stroke
@@
 	(hierarchical_label "GND"
 		(shape bidirectional)
-		(at 82.55 58.42 180)
+		(at 116.84 60.96 0)
+		(effects
+			(font
+				(size 1.27 1.27)
+			)
+			(justify left)
+		)
+	)
+	(hierarchical_label "Left_Fet"
+		(shape input)
+		(at 80.01 44.45 180)
 		(effects
 			(font
@@
 			)
 			(justify right)
-		)
-	)
-	(hierarchical_label "Left_Fet"
-		(shape input)
-		(at 119.38 48.26 0)
-		(effects
-			(font
-				(size 1.27 1.27)
-			)
-			(justify left)
 		)
 	)
 	(hierarchical_label "GND"
 		(shape bidirectional)
-		(at 82.55 45.72 180)
+		(at 116.84 48.26 0)
+		(effects
+			(font
+				(size 1.27 1.27)
+			)
+			(justify left)
+		)
+	)
+	(hierarchical_label "Head_fet"
+		(shape input)
+		(at 82.55 69.85 180)
 		(effects
 			(font
@@
 			)
 			(justify right)
-		)
-	)
-	(hierarchical_label "Head_fet"
-		(shape input)
-		(at 118.11 72.39 0)
-		(effects
-			(font
-				(size 1.27 1.27)
-			)
-			(justify left)
 		)
 	)
@@
 	(hierarchical_label "GND"
 		(shape bidirectional)
-		(at 81.28 69.85 180)
+		(at 118.11 72.39 0)
+		(effects
+			(font
+				(size 1.27 1.27)
+			)
+			(justify left)
+		)
+	)
+	(hierarchical_label "Right_Fet"
+		(shape input)
+		(at 81.28 58.42 180)
 		(effects
 			(font
@@
 			)
 			(justify right)
-		)
-	)
-	(hierarchical_label "Right_Fet"
-		(shape input)
-		(at 118.11 60.96 0)
-		(effects
-			(font
-				(size 1.27 1.27)
-			)
-			(justify left)
 		)
 	)
@@
 		)
 		(pin "FetIN" input
-			(at 110.49 48.26 0)
-			(effects
-				(font
-					(size 1.27 1.27)
-				)
-				(justify right)
+			(at 88.9 44.45 180)
+			(effects
+				(font
+					(size 1.27 1.27)
+				)
+				(justify left)
 			)
 		)
@@
 		)
 		(pin "GND" bidirectional
-			(at 88.9 45.72 180)
-			(effects
-				(font
-					(size 1.27 1.27)
-				)
-				(justify left)
+			(at 110.49 48.26 0)
+			(effects
+				(font
+					(size 1.27 1.27)
+				)
+				(justify right)
 			)
 		)
@@
 		)
 		(pin "FetIN" input
-			(at 110.49 72.39 0)
-			(effects
-				(font
-					(size 1.27 1.27)
-				)
-				(justify right)
+			(at 88.9 69.85 180)
+			(effects
+				(font
+					(size 1.27 1.27)
+				)
+				(justify left)
 			)
 		)
@@
 		)
 		(pin "GND" bidirectional
-			(at 88.9 69.85 180)
-			(effects
-				(font
-					(size 1.27 1.27)
-				)
-				(justify left)
+			(at 110.49 72.39 0)
+			(effects
+				(font
+					(size 1.27 1.27)
+				)
+				(justify right)
 			)
 		)
@@
 		)
 		(pin "FetIN" input
-			(at 110.49 60.96 0)
-			(effects
-				(font
-					(size 1.27 1.27)
-				)
-				(justify right)
+			(at 88.9 58.42 180)
+			(effects
+				(font
+					(size 1.27 1.27)
+				)
+				(justify left)
 			)
 		)
@@
 		)
 		(pin "GND" bidirectional
-			(at 88.9 58.42 180)
-			(effects
-				(font
-					(size 1.27 1.27)
-				)
-				(justify left)
-			)
-		)
+			(at 110.49 60.96 0)
+			(effects
+				(font
+					(size 1.27 1.27)
+				)
+				(justify right)
+			)
+		)

Commit message: footprint! mising 2
Changed lines of the file:
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@@
 	(wire
 		(pts
-			(xy 88.9 69.85) (xy 82.55 69.85)
+			(xy 82.55 69.85) (xy 88.9 69.85)
 		)
 		(stroke
@@
 	(wire
 		(pts
-			(xy 88.9 58.42) (xy 81.28 58.42)
-		)
-		(stroke
-			(width 0)
-			(type default)
-		)
-	)
-	(wire
-		(pts
 			(xy 116.84 60.96) (xy 110.49 60.96)
 		)
@@
 	(wire
 		(pts
-			(xy 110.49 69.85) (xy 118.11 69.85)
+			(xy 85.09 59.69) (xy 88.9 59.69)
+		)
+		(stroke
+			(width 0)
+			(type default)
+		)
+	)
+	(wire
+		(pts
+			(xy 110.49 69.85) (xy 115.57 69.85)
 		)
 		(stroke
@@
 	(wire
 		(pts
-			(xy 88.9 44.45) (xy 80.01 44.45)
+			(xy 85.09 45.72) (xy 88.9 45.72)
 		)
 		(stroke
@@
 	(hierarchical_label "Left_Fet"
 		(shape input)
-		(at 80.01 44.45 180)
-		(effects
-			(font
-				(size 1.27 1.27)
-			)
-			(justify right)
+		(at 119.38 45.72 0)
+		(effects
+			(font
+				(size 1.27 1.27)
+			)
+			(justify left)
 		)
 	)
@@
 	(hierarchical_label "Head_fet"
 		(shape input)
-		(at 82.55 69.85 180)
+		(at 115.57 69.85 0)
+		(effects
+			(font
+				(size 1.27 1.27)
+			)
+			(justify left)
+		)
+	)
+	(hierarchical_label "Right_Gate"
+		(shape input)
+		(at 85.09 59.69 180)
 		(effects
 			(font
@@
 			)
 			(justify right)
-		)
-	)
-	(hierarchical_label "Right_Gate"
-		(shape input)
-		(at 118.11 58.42 0)
-		(effects
-			(font
-				(size 1.27 1.27)
-			)
-			(justify left)
 		)
 	)
@@
 	(hierarchical_label "Right_Fet"
 		(shape input)
-		(at 81.28 58.42 180)
+		(at 118.11 58.42 0)
+		(effects
+			(font
+				(size 1.27 1.27)
+			)
+			(justify left)
+		)
+	)
+	(hierarchical_label "Head_Gate"
+		(shape input)
+		(at 82.55 69.85 180)
 		(effects
 			(font
@@
 		)
 	)
-	(hierarchical_label "Head_Gate"
-		(shape input)
-		(at 118.11 69.85 0)
-		(effects
-			(font
-				(size 1.27 1.27)
-			)
-			(justify left)
-		)
-	)
 	(hierarchical_label "Left_Gate"
 		(shape input)
-		(at 119.38 45.72 0)
-		(effects
-			(font
-				(size 1.27 1.27)
-			)
-			(justify left)
+		(at 85.09 45.72 180)
+		(effects
+			(font
+				(size 1.27 1.27)
+			)
+			(justify right)
 		)
 	)
@@
 		)
 		(pin "FetIN" input
-			(at 88.9 44.45 180)
+			(at 110.49 45.72 0)
+			(effects
+				(font
+					(size 1.27 1.27)
+				)
+				(justify right)
+			)
+		)
+		(pin "Gate" input
+			(at 88.9 45.72 180)
 			(effects
 				(font
@@
 				)
 				(justify left)
-			)
-		)
-		(pin "Gate" input
-			(at 110.49 45.72 0)
-			(effects
-				(font
-					(size 1.27 1.27)
-				)
-				(justify right)
 			)
 		)
@@
 		)
 		(pin "FetIN" input
+			(at 110.49 69.85 0)
+			(effects
+				(font
+					(size 1.27 1.27)
+				)
+				(justify right)
+			)
+		)
+		(pin "Gate" input
 			(at 88.9 69.85 180)
 			(effects
@@
 				)
 				(justify left)
-			)
-		)
-		(pin "Gate" input
-			(at 110.49 69.85 0)
-			(effects
-				(font
-					(size 1.27 1.27)
-				)
-				(justify right)
 			)
 		)
@@
 		)
 		(pin "FetIN" input
-			(at 88.9 58.42 180)
+			(at 110.49 58.42 0)
+			(effects
+				(font
+					(size 1.27 1.27)
+				)
+				(justify right)
+			)
+		)
+		(pin "Gate" input
+			(at 88.9 59.69 180)
 			(effects
 				(font
@@
 			)
 		)
-		(pin "Gate" input
-			(at 110.49 58.42 0)
-			(effects
-				(font
-					(size 1.27 1.27)
-				)
-				(justify right)
-			)
-		)
