File: hardware/PowerProtection.kicad_sch (KiCad schematic)
At the start: 18 parts, among them IC1 LM74502DDFR, Q1 PSMN012-100YS, Q2 PSMN012-100YS

Commit message: mcu and power
Changed lines of the file:
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@@
 	)
 	(hierarchical_label "GND"
-		(shape input)
+		(shape passive)
 		(at 60.96 68.58 270)
 		(effects
@@
 	)
 	(hierarchical_label "GND"
-		(shape input)
+		(shape passive)
 		(at 109.22 55.88 270)
 		(effects
@@
 	)
 	(hierarchical_label "GND"
-		(shape input)
+		(shape passive)
 		(at 139.7 95.25 270)
 		(effects
@@
 	)
 	(hierarchical_label "GND"
-		(shape input)
+		(shape passive)
 		(at 25.4 57.15 270)
 		(effects
@@
 	)
 	(hierarchical_label "GND"
-		(shape input)
+		(shape passive)
 		(at 74.93 99.06 270)
 		(effects
@@
 	)
 	(hierarchical_label "GND"
-		(shape input)
+		(shape passive)
 		(at 129.54 95.25 270)
 		(effects
@@
 	)
 	(hierarchical_label "GND"
-		(shape input)
+		(shape passive)
 		(at 120.65 95.25 270)
 		(effects
@@
 	)
 	(hierarchical_label "GND"
-		(shape input)
+		(shape passive)
 		(at 34.29 57.15 270)
 		(effects
@@
 	)
 	(hierarchical_label "GND"
-		(shape input)
+		(shape passive)
 		(at 110.49 95.25 270)
 		(effects
@@
 	)
 	(hierarchical_label "GND"
-		(shape input)
+		(shape passive)
 		(at 35.56 88.9 270)
 		(effects
@@
 	)
 	(hierarchical_label "GND"
-		(shape input)
+		(shape passive)
 		(at 43.18 88.9 270)
 		(effects

Commit message: someone please check if i fucked up removing boot
Changed lines of the file:
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@@
 	)
 	(hierarchical_label "GND"
-		(shape passive)
+		(shape bidirectional)
 		(at 60.96 68.58 270)
 		(effects
@@
 	)
 	(hierarchical_label "GND"
-		(shape passive)
+		(shape bidirectional)
 		(at 109.22 55.88 270)
 		(effects
@@
 	)
 	(hierarchical_label "GND"
-		(shape passive)
+		(shape bidirectional)
 		(at 139.7 95.25 270)
 		(effects
@@
 	)
 	(hierarchical_label "GND"
-		(shape passive)
+		(shape bidirectional)
 		(at 25.4 57.15 270)
 		(effects
@@
 	)
 	(hierarchical_label "GND"
-		(shape passive)
+		(shape bidirectional)
 		(at 74.93 99.06 270)
 		(effects
@@
 	)
 	(hierarchical_label "GND"
-		(shape passive)
+		(shape bidirectional)
 		(at 129.54 95.25 270)
 		(effects
@@
 	)
 	(hierarchical_label "GND"
-		(shape passive)
+		(shape bidirectional)
 		(at 120.65 95.25 270)
 		(effects
@@
 	)
 	(hierarchical_label "GND"
-		(shape passive)
+		(shape bidirectional)
 		(at 34.29 57.15 270)
 		(effects
@@
 	)
 	(hierarchical_label "GND"
-		(shape passive)
+		(shape bidirectional)
 		(at 110.49 95.25 270)
 		(effects
@@
 	)
 	(hierarchical_label "GND"
-		(shape passive)
+		(shape bidirectional)
 		(at 35.56 88.9 270)
 		(effects
@@
 	)
 	(hierarchical_label "GND"
-		(shape passive)
+		(shape bidirectional)
 		(at 43.18 88.9 270)
 		(effects

Commit message: rawr
Parts:
- IC1: Manufacturer_Name Texas Instruments -> (none); Manufacturer_Part_Number LM74502DDFR -> (none); Mouser Part Number 595-LM74502DDFR -> (none); Mouser Price/Stock https://www.mouser.co.uk/ProductDetail/Texas-Instruments/LM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 -> (none)
- R10: renamed from R23; symbol Device:R_US -> Device:R
- R11: renamed from R24; symbol Device:R_US -> Device:R
- R3: renamed from R19; symbol Device:R_US -> Device:R
- R4: renamed from R20; symbol Device:R_US -> Device:R; Mouser Part Number 594-MCT06030C3309FP5 -> (none)
- R5: renamed from R21; symbol Device:R_US -> Device:R
- R6: renamed from R22; symbol Device:R_US -> Device:R
- renumbered C27 to C1, C28 to C2, C29 to C3, C30 to C4, C31 to C5, C32 to C6, C33 to C7, D10 to D1, D11 to D2
Other:
- note added: "Supp Battery Range: 10V-14.7V"

Commit message: footprint! mising 2
Parts:
- renumbered C1 to C2, C2 to C3, C3 to C4, C4 to C5, C5 to C6, C6 to C7, C7 to C8, D1 to D3, D2 to D4, Q1 to Q2, Q2 to Q3, R6 to R10, R10 to R11, R11 to R12, R3 to R7, R4 to R8, R5 to R9
Changed lines of the file:
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@@
 		(in_pos_files yes)
 		(dnp no)
-		(property "Reference" "D2"
+		(property "Reference" "D4"
 			(at 40.64 82.296 0)
 			(show_name no)
@@
 			(project "DEI"
 				(path "/1469f349-54e5-4a37-953e-ac48c70e29b2/d41a835d-0002-40e6-b2c5-562251bf7d32/63920d64-0484-425f-8f64-1c9300ee1a5c"
-					(reference "D2")
+					(reference "D4")
 					(unit 1)
 				)
@@
 		(dnp no)
 		(fields_autoplaced yes)
-		(property "Reference" "C3"
+		(property "Reference" "C4"
 			(at 57.785 80.0099 0)
 			(show_name no)
@@
 			(project "DEI"
 				(path "/1469f349-54e5-4a37-953e-ac48c70e29b2/d41a835d-0002-40e6-b2c5-562251bf7d32/63920d64-0484-425f-8f64-1c9300ee1a5c"
-					(reference "C3")
+					(reference "C4")
 					(unit 1)
 				)
@@
 		(in_pos_files yes)
 		(dnp no)
-		(property "Reference" "D1"
+		(property "Reference" "D3"
 			(at 22.606 49.276 0)
 			(show_name no)
@@
 			(project "DEI"
 				(path "/1469f349-54e5-4a37-953e-ac48c70e29b2/d41a835d-0002-40e6-b2c5-562251bf7d32/63920d64-0484-425f-8f64-1c9300ee1a5c"
-					(reference "D1")
+					(reference "D3")
 					(unit 1)
 				)
@@
 		(dnp no)
 		(fields_autoplaced yes)
-		(property "Reference" "R3"
+		(property "Reference" "R7"
 			(at 45.72 60.9599 0)
 			(show_name no)
@@
 			(project "DEI"
 				(path "/1469f349-54e5-4a37-953e-ac48c70e29b2/d41a835d-0002-40e6-b2c5-562251bf7d32/63920d64-0484-425f-8f64-1c9300ee1a5c"
-					(reference "R3")
+					(reference "R7")
 					(unit 1)
 				)
@@
 		(in_pos_files yes)
 		(dnp no)
-		(property "Reference" "R11"
+		(property "Reference" "R12"
 			(at 137.668 90.17 90)
 			(show_name no)
@@
 			(project "DEI"
 				(path "/1469f349-54e5-4a37-953e-ac48c70e29b2/d41a835d-0002-40e6-b2c5-562251bf7d32/63920d64-0484-425f-8f64-1c9300ee1a5c"
-					(reference "R11")
+					(reference "R12")
 					(unit 1)
 				)
@@
 		(in_pos_files yes)
 		(dnp no)
-		(property "Reference" "C1"
+		(property "Reference" "C2"
 			(at 38.1 49.5299 0)
 			(show_name no)
@@
 			(project "DEI"
 				(path "/1469f349-54e5-4a37-953e-ac48c70e29b2/d41a835d-0002-40e6-b2c5-562251bf7d32/63920d64-0484-425f-8f64-1c9300ee1a5c"
-					(reference "C1")
+					(reference "C2")
 					(unit 1)
 				)
@@
 		(in_pos_files yes)
 		(dnp no)
-		(property "Reference" "R4"
+		(property "Reference" "R8"
 			(at 67.31 54.61 90)
 			(show_name no)
@@
 			(project "DEI"
 				(path "/1469f349-54e5-4a37-953e-ac48c70e29b2/d41a835d-0002-40e6-b2c5-562251bf7d32/63920d64-0484-425f-8f64-1c9300ee1a5c"
-					(reference "R4")
+					(reference "R8")
 					(unit 1)
 				)
@@
 		(in_pos_files yes)
 		(dnp no)
-		(property "Reference" "Q1"
+		(property "Reference" "Q2"
 			(at 52.578 38.862 90)
 			(show_name no)
@@
 			(project "DEI"
 				(path "/1469f349-54e5-4a37-953e-ac48c70e29b2/d41a835d-0002-40e6-b2c5-562251bf7d32/63920d64-0484-425f-8f64-1c9300ee1a5c"
-					(reference "Q1")
+					(reference "Q2")
 					(unit 1)
 				)
@@
 		(in_pos_files yes)
 		(dnp no)
-		(property "Reference" "C6"
+		(property "Reference" "C7"
 			(at 113.284 89.154 0)
 			(show_name no)
@@
 			(project "DEI"
 				(path "/1469f349-54e5-4a37-953e-ac48c70e29b2/d41a835d-0002-40e6-b2c5-562251bf7d32/63920d64-0484-425f-8f64-1c9300ee1a5c"
-					(reference "C6")
+					(reference "C7")
 					(unit 1)
 				)
@@
 		(in_pos_files yes)
 		(dnp no)
-		(property "Reference" "C4"
+		(property "Reference" "C5"
 			(at 54.864 62.23 0)
 			(show_name no)
@@
 			(project "DEI"
 				(path "/1469f349-54e5-4a37-953e-ac48c70e29b2/d41a835d-0002-40e6-b2c5-562251bf7d32/63920d64-0484-425f-8f64-1c9300ee1a5c"
-					(reference "C4")
+					(reference "C5")
 					(unit 1)
 				)
@@
 		(in_pos_files yes)
 		(dnp no)
-		(property "Reference" "C5"
+		(property "Reference" "C6"
 			(at 112.395 49.5299 0)
 			(show_name no)
@@
 			(project "DEI"
 				(path "/1469f349-54e5-4a37-953e-ac48c70e29b2/d41a835d-0002-40e6-b2c5-562251bf7d32/63920d64-0484-425f-8f64-1c9300ee1a5c"
-					(reference "C5")
+					(reference "C6")
 					(unit 1)
 				)
@@
 		(in_pos_files yes)
 		(dnp no)
-		(property "Reference" "Q2"
+		(property "Reference" "Q3"
 			(at 100.584 38.608 90)
 			(show_name no)
@@
 			(project "DEI"
 				(path "/1469f349-54e5-4a37-953e-ac48c70e29b2/d41a835d-0002-40e6-b2c5-562251bf7d32/63920d64-0484-425f-8f64-1c9300ee1a5c"
-					(reference "Q2")
+					(reference "Q3")
 					(unit 1)
 				)
@@
 		(in_pos_files yes)
 		(dnp no)
-		(property "Reference" "R6"
+		(property "Reference" "R10"
 			(at 118.618 90.424 90)
 			(show_name no)
@@
 			(project "DEI"
 				(path "/1469f349-54e5-4a37-953e-ac48c70e29b2/d41a835d-0002-40e6-b2c5-562251bf7d32/63920d64-0484-425f-8f64-1c9300ee1a5c"
-					(reference "R6")
+					(reference "R10")
 					(unit 1)
 				)
@@
 		(in_pos_files yes)
 		(dnp no)
-		(property "Reference" "C2"
+		(property "Reference" "C3"
 			(at 31.75 82.5499 0)
 			(show_name no)
@@
 			(project "DEI"
 				(path "/1469f349-54e5-4a37-953e-ac48c70e29b2/d41a835d-0002-40e6-b2c5-562251bf7d32/63920d64-0484-425f-8f64-1c9300ee1a5c"
-					(reference "C2")
+					(reference "C3")
 					(unit 1)
 				)
@@
 		(in_pos_files yes)
 		(dnp no)
-		(property "Reference" "C7"
+		(property "Reference" "C8"
 			(at 132.08 88.9 0)
 			(show_name no)
@@
 			(project "DEI"
 				(path "/1469f349-54e5-4a37-953e-ac48c70e29b2/d41a835d-0002-40e6-b2c5-562251bf7d32/63920d64-0484-425f-8f64-1c9300ee1a5c"
-					(reference "C7")
+					(reference "C8")
 					(unit 1)
 				)
@@
 		(in_pos_files yes)
 		(dnp no)
-		(property "Reference" "R5"
+		(property "Reference" "R9"
 			(at 118.11 78.74 90)
 			(show_name no)
@@
 			(project "DEI"
 				(path "/1469f349-54e5-4a37-953e-ac48c70e29b2/d41a835d-0002-40e6-b2c5-562251bf7d32/63920d64-0484-425f-8f64-1c9300ee1a5c"
-					(reference "R5")
+					(reference "R9")
 					(unit 1)
 				)
@@
 		(in_pos_files yes)
 		(dnp no)
-		(property "Reference" "R10"
+		(property "Reference" "R11"
 			(at 137.16 77.47 90)
 			(show_name no)
@@
 			(project "DEI"
 				(path "/1469f349-54e5-4a37-953e-ac48c70e29b2/d41a835d-0002-40e6-b2c5-562251bf7d32/63920d64-0484-425f-8f64-1c9300ee1a5c"
-					(reference "R10")
-					(unit 1)
-				)
+					(reference "R11")
+					(unit 1)
+				)
