File: hardware/Power_Mux.kicad_sch (KiCad schematic)
At the start: 6 parts, among them U5 TPS2117DRLR

Commit message: rawr
Parts:
- C16: renamed from C34; value 0.1uF -> 0.1u; Mfg MLASH168SB7104KTNA01 -> (none)
- C17: renamed from C35; value 0.1uF -> 0.1u; Mfg MLASH168SB7104KTNA01 -> (none)
- C19: renamed from C36; value 0.1uF -> 0.1u; Mfg MLASH168SB7104KTNA01 -> (none)
- C20: renamed from C37; value 0.1uF -> 0.1u; Mfg MLASH168SB7104KTNA01 -> (none)
- U2: renamed from U5; MANUFACTURER Texas Instruments -> (none); MAXIMUM_PACKAGE_HEIGHT 0.6mm -> (none); PARTREV A -> (none); STANDARD IPC-7351B -> (none)
- renumbered R27 to R14
Changed lines of the file:
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@@
 		(in_pos_files yes)
 		(dnp no)
-		(property "Reference" "C37"
+		(property "Reference" "C20"
 			(at 91.8972 57.2516 0)
 			(show_name no)
@@
 			)
 		)
-		(property "Value" "0.1uF"
+		(property "Value" "0.1u"
 			(at 91.8972 59.563 0)
 			(show_name no)
@@
 			)
 		)
-		(property "Mfg" "MLASH168SB7104KTNA01"
-			(at 88.9 58.42 0)
-			(hide yes)
-			(show_name no)
-			(do_not_autoplace no)
-			(effects
-				(font
-					(size 1.27 1.27)
-				)
-			)
-		)
 		(pin "1"
 		)
@@
 		(instances
 			(project "DEI"
-				(path "/1469f349-54e5-4a37-953e-ac48c70e29b2/d41a835d-0002-40e6-b2c5-562251bf7d32/7b8754e3-7888-44e1-99a1-5ee65bae4b91"
-					(reference "C37")
-					(unit 1)
-				)
-			)
-			(project "power-mux-block"
+				(path "/1469f349-54e5-4a37-953e-ac48c70e29b2/d41a835d-0002-40e6-b2c5-562251bf7d32/b8ad50d8-c271-44ff-b140-dd0f61fc62a8"
+					(reference "C20")
+					(unit 1)
+				)
+			)
+			(project "Power_Mux"
 				(path "/c8207045-8aef-4538-bcc4-1e380c549c2c"
 					(reference "C4")
@@
 		(in_pos_files yes)
 		(dnp no)
-		(property "Reference" "R27"
+		(property "Reference" "R14"
 			(at 78.994 67.564 0)
 			(show_name no)
@@
 		(instances
 			(project "DEI"
-				(path "/1469f349-54e5-4a37-953e-ac48c70e29b2/d41a835d-0002-40e6-b2c5-562251bf7d32/7b8754e3-7888-44e1-99a1-5ee65bae4b91"
-					(reference "R27")
-					(unit 1)
-				)
-			)
-			(project "power-mux-block"
+				(path "/1469f349-54e5-4a37-953e-ac48c70e29b2/d41a835d-0002-40e6-b2c5-562251bf7d32/b8ad50d8-c271-44ff-b140-dd0f61fc62a8"
+					(reference "R14")
+					(unit 1)
+				)
+			)
+			(project "Power_Mux"
 				(path "/c8207045-8aef-4538-bcc4-1e380c549c2c"
 					(reference "R1")
@@
 		(in_pos_files yes)
 		(dnp no)
-		(property "Reference" "C34"
+		(property "Reference" "C16"
 			(at 24.5872 44.5516 0)
 			(show_name no)
@@
 			)
 		)
-		(property "Value" "0.1uF"
+		(property "Value" "0.1u"
 			(at 24.5872 46.863 0)
 			(show_name no)
@@
 			)
 		)
-		(property "Mfg" "MLASH168SB7104KTNA01"
-			(at 21.59 45.72 0)
-			(hide yes)
-			(show_name no)
-			(do_not_autoplace no)
-			(effects
-				(font
-					(size 1.27 1.27)
-				)
-			)
-		)
 		(pin "1"
 		)
@@
 		(instances
 			(project "DEI"
-				(path "/1469f349-54e5-4a37-953e-ac48c70e29b2/d41a835d-0002-40e6-b2c5-562251bf7d32/7b8754e3-7888-44e1-99a1-5ee65bae4b91"
-					(reference "C34")
-					(unit 1)
-				)
-			)
-			(project "power-mux-block"
+				(path "/1469f349-54e5-4a37-953e-ac48c70e29b2/d41a835d-0002-40e6-b2c5-562251bf7d32/b8ad50d8-c271-44ff-b140-dd0f61fc62a8"
+					(reference "C16")
+					(unit 1)
+				)
+			)
+			(project "Power_Mux"
 				(path "/c8207045-8aef-4538-bcc4-1e380c549c2c"
 					(reference "C1")
@@
 		(dnp no)
 		(fields_autoplaced yes)
-		(property "Reference" "U5"
+		(property "Reference" "U2"
 			(at 60.96 44.45 0)
 			(show_name no)
@@
 			)
 		)
-		(property "PARTREV" "A"
-			(at 60.96 62.23 0)
-			(hide yes)
-			(show_name no)
-			(do_not_autoplace no)
-			(effects
-				(font
-					(size 1.27 1.27)
-				)
-				(justify bottom)
-			)
-		)
-		(property "STANDARD" "IPC-7351B"
-			(at 60.96 62.23 0)
-			(hide yes)
-			(show_name no)
-			(do_not_autoplace no)
-			(effects
-				(font
-					(size 1.27 1.27)
-				)
-				(justify bottom)
-			)
-		)
-		(property "MAXIMUM_PACKAGE_HEIGHT" "0.6mm"
-			(at 60.96 62.23 0)
-			(hide yes)
-			(show_name no)
-			(do_not_autoplace no)
-			(effects
-				(font
-					(size 1.27 1.27)
-				)
-				(justify bottom)
-			)
-		)
-		(property "MANUFACTURER" "Texas Instruments"
-			(at 60.96 62.23 0)
-			(hide yes)
-			(show_name no)
-			(do_not_autoplace no)
-			(effects
-				(font
-					(size 1.27 1.27)
-				)
-				(justify bottom)
-			)
-		)
 		(property "P/N" "TPS2117DRLR"
 			(at 60.96 49.53 0)
@@
 		(instances
 			(project "DEI"
-				(path "/1469f349-54e5-4a37-953e-ac48c70e29b2/d41a835d-0002-40e6-b2c5-562251bf7d32/7b8754e3-7888-44e1-99a1-5ee65bae4b91"
-					(reference "U5")
-					(unit 1)
-				)
-			)
-			(project ""
+				(path "/1469f349-54e5-4a37-953e-ac48c70e29b2/d41a835d-0002-40e6-b2c5-562251bf7d32/b8ad50d8-c271-44ff-b140-dd0f61fc62a8"
+					(reference "U2")
+					(unit 1)
+				)
+			)
+			(project "Power_Mux"
 				(path "/c8207045-8aef-4538-bcc4-1e380c549c2c"
 					(reference "U1")
@@
 		(in_pos_files yes)
 		(dnp no)
-		(property "Reference" "C36"
+		(property "Reference" "C19"
 			(at 42.3672 67.4116 0)
 			(show_name no)
@@
 			)
 		)
-		(property "Value" "0.1uF"
+		(property "Value" "0.1u"
 			(at 42.3672 69.723 0)
 			(show_name no)
@@
 			)
 		)
-		(property "Mfg" "MLASH168SB7104KTNA01"
-			(at 39.37 68.58 0)
-			(hide yes)
-			(show_name no)
-			(do_not_autoplace no)
-			(effects
-				(font
-					(size 1.27 1.27)
-				)
-			)
-		)
 		(pin "1"
 		)
@@
 		(instances
 			(project "DEI"
-				(path "/1469f349-54e5-4a37-953e-ac48c70e29b2/d41a835d-0002-40e6-b2c5-562251bf7d32/7b8754e3-7888-44e1-99a1-5ee65bae4b91"
-					(reference "C36")
-					(unit 1)
-				)
-			)
-			(project "power-mux-block"
+				(path "/1469f349-54e5-4a37-953e-ac48c70e29b2/d41a835d-0002-40e6-b2c5-562251bf7d32/b8ad50d8-c271-44ff-b140-dd0f61fc62a8"
+					(reference "C19")
+					(unit 1)
+				)
+			)
+			(project "Power_Mux"
 				(path "/c8207045-8aef-4538-bcc4-1e380c549c2c"
 					(reference "C3")
@@
 		(in_pos_files yes)
 		(dnp no)
-		(property "Reference" "C35"
+		(property "Reference" "C17"
 			(at 38.5572 44.5516 0)
 			(show_name no)
@@
 			)
 		)
-		(property "Value" "0.1uF"
+		(property "Value" "0.1u"
 			(at 38.5572 46.863 0)
 			(show_name no)
@@
 			)
 		)
-		(property "Mfg" "MLASH168SB7104KTNA01"
-			(at 35.56 45.72 0)
-			(hide yes)
-			(show_name no)
-			(do_not_autoplace no)
-			(effects
-				(font
-					(size 1.27 1.27)
-				)
-			)
-		)
 		(pin "1"
 		)
@@
 		(instances
 			(project "DEI"
-				(path "/1469f349-54e5-4a37-953e-ac48c70e29b2/d41a835d-0002-40e6-b2c5-562251bf7d32/7b8754e3-7888-44e1-99a1-5ee65bae4b91"
-					(reference "C35")
-					(unit 1)
-				)
-			)
-			(project "power-mux-block"
+				(path "/1469f349-54e5-4a37-953e-ac48c70e29b2/d41a835d-0002-40e6-b2c5-562251bf7d32/b8ad50d8-c271-44ff-b140-dd0f61fc62a8"
+					(reference "C17")
+					(unit 1)
+				)
+			)
+			(project "Power_Mux"
 				(path "/c8207045-8aef-4538-bcc4-1e380c549c2c"
 					(reference "C2")

Commit message: footprint! mising 2
Parts:
- renumbered C19 to C18, C20 to C19, R14 to R17
Changed lines of the file:
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@@
 		(in_pos_files yes)
 		(dnp no)
-		(property "Reference" "C20"
+		(property "Reference" "C19"
 			(at 91.8972 57.2516 0)
 			(show_name no)
@@
 			(project "DEI"
 				(path "/1469f349-54e5-4a37-953e-ac48c70e29b2/d41a835d-0002-40e6-b2c5-562251bf7d32/b8ad50d8-c271-44ff-b140-dd0f61fc62a8"
-					(reference "C20")
+					(reference "C19")
 					(unit 1)
 				)
@@
 		(in_pos_files yes)
 		(dnp no)
-		(property "Reference" "R14"
+		(property "Reference" "R17"
 			(at 78.994 67.564 0)
 			(show_name no)
@@
 			(project "DEI"
 				(path "/1469f349-54e5-4a37-953e-ac48c70e29b2/d41a835d-0002-40e6-b2c5-562251bf7d32/b8ad50d8-c271-44ff-b140-dd0f61fc62a8"
-					(reference "R14")
+					(reference "R17")
 					(unit 1)
 				)
@@
 		(in_pos_files yes)
 		(dnp no)
-		(property "Reference" "C19"
+		(property "Reference" "C18"
 			(at 42.3672 67.4116 0)
 			(show_name no)
@@
 			(project "DEI"
 				(path "/1469f349-54e5-4a37-953e-ac48c70e29b2/d41a835d-0002-40e6-b2c5-562251bf7d32/b8ad50d8-c271-44ff-b140-dd0f61fc62a8"
-					(reference "C19")
-					(unit 1)
-				)
+					(reference "C18")
+					(unit 1)
+				)
